File: subsheet_102.sch (KiCad schematic (older format))
At the start: 7 parts, among them U102 EPROM_32_PINS_DIP_PHY, U103 EPROM_32_PINS_DIP_PHY

Commit message: Resolves #8 : Assign 1206 hand-solder footprints to non polarized capacitors
Parts:
- C113, C114: footprint commons_passives_THT:Passive_THT_capacitor_mlcc_W2.54mm_L7.62mm -> Capacitor_SMD:C_1206_3216Metric_Pad1.33x1.80mm_HandSolder
Changed lines of the file:
@@
 F 0 "C113" H 1425 3600 50  0000 L CNN
 F 1 "0.1uF" H 1425 3400 50  0000 L CNN
-F 2 "commons_passives_THT:Passive_THT_capacitor_mlcc_W2.54mm_L7.62mm" H 1438 3350 50  0001 C CNN
+F 2 "Capacitor_SMD:C_1206_3216Metric_Pad1.33x1.80mm_HandSolder" H 1438 3350 50  0001 C CNN
 F 3 "~" H 1400 3500 50  0001 C CNN
 	1    1400 3500
@@
 F 0 "C114" H 6925 3600 50  0000 L CNN
 F 1 "0.1uF" H 6925 3400 50  0000 L CNN
-F 2 "commons_passives_THT:Passive_THT_capacitor_mlcc_W2.54mm_L7.62mm" H 6938 3350 50  0001 C CNN
+F 2 "Capacitor_SMD:C_1206_3216Metric_Pad1.33x1.80mm_HandSolder" H 6938 3350 50  0001 C CNN
 F 3 "~" H 6900 3500 50  0001 C CNN
 	1    6900 3500
