File: subsheet_106.sch (KiCad schematic (older format))
At the start: 47 parts, among them Q100 2N3904, Q101 2N3904, Q102 2N3904, Q103 2N3904, Q104 2N3904, U402 32.215905 MHz (NTSC) — 32.084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, Y100 4.433618MHz, Y101 32.084988MHz

Commit message: Delete circuitry related to PAL/NTSC and modulator
Parts:
- removed C115: 4700pF, commons_passives_THT:Passive_THT_capacitor_W2.54mm_L10.16mm, symbol Device:C
- removed C116: 0.47uF, commons_passives_THT:Passive_THT_capacitor_mlcc_W2.54mm_L10.16mm, symbol Device:C
- removed C117: 2.7–10pF, commons_passives_THT:Passive_THT_variable_capacitor_rad_D7.62mm_P5.08mm, symbol Device:C_Variable
- removed C118: 8.2pF, commons_passives_THT:Passive_THT_capacitor_W2.54mm_L12.70mm, symbol Device:C
- removed C119: 470pF, commons_passives_THT:Passive_THT_capacitor_W2.54mm_L12.70mm, symbol Device:C
- removed C120: 1000pF, commons_passives_THT:Passive_THT_capacitor_W2.54mm_L12.70mm, symbol Device:C
- removed C121: 100pF, commons_passives_THT:Passive_THT_capacitor_W2.54mm_L10.16mm, symbol Device:C
- removed C122: 220pF, commons_passives_THT:Passive_THT_capacitor_W2.54mm_L12.70mm, symbol Device:C
- removed C123, C128: 1000pF, commons_passives_THT:Passive_THT_capacitor_W2.54mm_L10.16mm, symbol Device:C
- removed C124: 22nF, commons_passives_THT:Passive_THT_capacitor_W2.54mm_L10.16mm, symbol Device:C
- removed C125: 8.2pF, commons_passives_THT:Passive_THT_capacitor_W2.54mm_L10.16mm, symbol Device:C
- removed C126: 33pF, commons_passives_THT:Passive_THT_capacitor_W2.54mm_L10.16mm, symbol Device:C
- removed C127: 68pF, commons_passives_THT:Passive_THT_capacitor_W2.54mm_L10.16mm, symbol Device:C
- removed C129: 27pF, commons_passives_THT:Passive_THT_capacitor_W2.54mm_L10.16mm, symbol Device:C
- removed D101, D102: 1SV69, commons_passives_THT:Passive_THT_diode_W2.54mm_L12.70mm, symbol Device:D_Capacitance
- removed L101: 0.27uH, commons_passives_THT:Passive_THT_inductor_W5.08mm_L15.24mm, symbol Device:L_Small
- removed L102: 1.5uH, commons_passives_THT:Passive_THT_inductor_W5.08mm_L15.24mm, symbol Device:L
- removed L103: 1uH, commons_passives_THT:Passive_THT_inductor_W5.08mm_L15.24mm, symbol Device:L_Small
- removed Q100, Q101, Q102, Q103, Q104: 2N3904, Package_TO_SOT_THT:TO-92_Inline_Wide, symbol Device:Q_NPN_EBC
- removed R113: 22K, commons_passives_THT:Passive_THT_resistor_W2.54mm_L12.70mm, symbol Device:R_Small_US
- removed R114: 10K, commons_passives_THT:Passive_THT_resistor_W2.54mm_L12.70mm, symbol Device:R_Small_US
- removed R115, R118: 1K, commons_passives_THT:Passive_THT_resistor_W2.54mm_L12.70mm, symbol Device:R_Small_US
- removed R116: 18K, commons_passives_THT:Passive_THT_resistor_W2.54mm_L12.70mm, symbol Device:R_Small_US
- removed R117: 2K4, commons_passives_THT:Passive_THT_resistor_W2.54mm_L12.70mm, symbol Device:R_Small_US
- removed R119: 2K2, commons_passives_THT:Passive_THT_resistor_W2.54mm_L12.70mm, symbol Device:R_US
- removed R120: 2K2, commons_passives_THT:Passive_THT_resistor_W2.54mm_L12.70mm, symbol Device:R_Small_US
- removed R121, R122: 100K, commons_passives_THT:Passive_THT_resistor_W2.54mm_L12.70mm, symbol Device:R_Small_US
- removed R123: 4K7, commons_passives_THT:Passive_THT_resistor_W2.54mm_L12.70mm, symbol Device:R_US
- removed R124: 6K8, commons_passives_THT:Passive_THT_resistor_W2.54mm_L12.70mm, symbol Device:R_Small_US
- removed R125: 5K6, commons_passives_THT:Passive_THT_resistor_W2.54mm_L12.70mm, symbol Device:R_Small_US
- removed R126: 560, commons_passives_THT:Passive_THT_resistor_W2.54mm_L12.70mm, symbol Device:R_Small_US
- removed R127: 430, commons_passives_THT:Passive_THT_resistor_W2.54mm_L12.70mm, symbol Device:R_Small_US
- removed R128: 2K7, commons_passives_THT:Passive_THT_resistor_W2.54mm_L12.70mm, symbol Device:R_Small_US
- removed R129: 3K6, commons_passives_THT:Passive_THT_resistor_W2.54mm_L12.70mm, symbol Device:R_Small_US
- removed R130: 150, commons_passives_THT:Passive_THT_resistor_W2.54mm_L12.70mm, symbol Device:R_Small_US
- removed Y100: 4.433618MHz, Crystal:Crystal_HC18-U_Horizontal, symbol Device:Crystal
- removed Y101: 32.084988MHz, Crystal:Crystal_HC18-U_Horizontal, symbol Device:Crystal
Connections:
- net labels removed: CCLK, G12V, LINE_PHASE, VLL
- wire segments 122 -> 5
Other:
- note removed: "Diode 1SV69 : Electronic tuning for UHF/VHF TV Tuner\nhttps://pdf1.alldatasheet.com/datasheet-pdf/view/107651/ETC/1SV69.html"
- note removed: "From U306"
- note removed: "From \nU204"
- note removed: "Generation of 32 MHz clock (32MHZ)"
- note removed: "Generation of Pal sub-Carrier CLocK (CCLK)"
- note removed: "Installed ONLY in PAL systems"
- note removed: "To U306\nand U403"
- note removed: "To have an idea of what this circuitry is for, see https://en.wikipedia.org/wiki/PAL"

Commit message: Resolves #8 : Assign 1206 hand-solder footprints to non polarized capacitors
Parts:
- C409: footprint commons_passives_THT:Passive_THT_capacitor_mlcc_W2.54mm_L7.62mm -> Capacitor_SMD:C_1206_3216Metric_Pad1.33x1.80mm_HandSolder
Changed lines of the file:
@@
 F 0 "C409" H 3275 2350 50  0000 L CNN
 F 1 "100pF" H 3275 2150 50  0000 L CNN
-F 2 "commons_passives_THT:Passive_THT_capacitor_mlcc_W2.54mm_L7.62mm" H 3288 2100 50  0001 C CNN
+F 2 "Capacitor_SMD:C_1206_3216Metric_Pad1.33x1.80mm_HandSolder" H 3288 2100 50  0001 C CNN
 F 3 "~" H 3250 2250 50  0001 C CNN
 	1    3250 2250
