File: subsheet_202.sch (KiCad schematic (older format))
At the start: 15 parts, among them J203 DB-25S Parallel port, U202 YM2149_PHY

Commit message: Removed T-filters
Parts:
- removed L209, L210, L211, L212, L213, L214, L215, L216, L217, L218: EMI_Filter_LCL, commons_passives_THT:Passive_THT_EMI_filter_W5.08mm_L7.62mm, symbol Device:EMI_Filter_LCL
Connections:
- net labels removed: parallel1, parallel11, parallel2, parallel3, parallel4, parallel5, parallel6, parallel7, parallel8, parallel9
- wire segments 91 -> 71
Other:
- moved on the sheet: R212

Commit message: Resolves #13 : assign 1206 hand-solder footprints to resistors
Parts:
- R212, R220: footprint commons_passives_THT:Passive_THT_resistor_W2.54mm_L12.70mm -> Resistor_SMD:R_1206_3216Metric_Pad1.30x1.75mm_HandSolder
Changed lines of the file:
@@
 F 0 "R220" V 2700 2550 50  0000 C CNN
 F 1 "1K" V 2900 2550 50  0000 C CNN
-F 2 "commons_passives_THT:Passive_THT_resistor_W2.54mm_L12.70mm" H 2800 2550 50  0001 C CNN
+F 2 "Resistor_SMD:R_1206_3216Metric_Pad1.30x1.75mm_HandSolder" H 2800 2550 50  0001 C CNN
 F 3 "~" H 2800 2550 50  0001 C CNN
 	1    2800 2550
@@
 F 0 "R212" H 4300 5900 50  0000 C CNN
 F 1 "3K3" H 4300 5800 50  0000 C CNN
-F 2 "commons_passives_THT:Passive_THT_resistor_W2.54mm_L12.70mm" H 4150 5850 50  0001 C CNN
+F 2 "Resistor_SMD:R_1206_3216Metric_Pad1.30x1.75mm_HandSolder" H 4150 5850 50  0001 C CNN
 F 3 "~" H 4150 5850 50  0001 C CNN
 	1    4150 5850

Commit message: Resolves #8 : Assign 1206 hand-solder footprints to non polarized capacitors
Parts:
- C214: footprint commons_passives_THT:Passive_THT_capacitor_mlcc_W2.54mm_L7.62mm -> Capacitor_SMD:C_1206_3216Metric_Pad1.33x1.80mm_HandSolder
Changed lines of the file:
@@
 F 0 "C214" H 5825 2100 50  0000 L CNN
 F 1 "0.1uF" H 5825 1900 50  0000 L CNN
-F 2 "commons_passives_THT:Passive_THT_capacitor_mlcc_W2.54mm_L7.62mm" H 5838 1850 50  0001 C CNN
+F 2 "Capacitor_SMD:C_1206_3216Metric_Pad1.33x1.80mm_HandSolder" H 5838 1850 50  0001 C CNN
 F 3 "~" H 5800 2000 50  0001 C CNN
 	1    5800 2000
