File: subsheet_303.sch (KiCad schematic (older format))
At the start: 4 parts, among them U303 8.010613 MHz, U304 74LS74_PHY

Commit message: Resolves #8 : Assign 1206 hand-solder footprints to non polarized capacitors
Parts:
- C300, C301: footprint commons_passives_THT:Passive_THT_capacitor_mlcc_W2.54mm_L7.62mm -> Capacitor_SMD:C_1206_3216Metric_Pad1.33x1.80mm_HandSolder
Changed lines of the file:
@@
 F 0 "C300" H 6575 1800 50  0000 L CNN
 F 1 "0.1uF" H 6575 1600 50  0000 L CNN
-F 2 "commons_passives_THT:Passive_THT_capacitor_mlcc_W2.54mm_L7.62mm" H 6588 1550 50  0001 C CNN
+F 2 "Capacitor_SMD:C_1206_3216Metric_Pad1.33x1.80mm_HandSolder" H 6588 1550 50  0001 C CNN
 F 3 "~" H 6550 1700 50  0001 C CNN
 	1    6550 1700
@@
 F 0 "C301" H 1575 1700 50  0000 L CNN
 F 1 "0.1uF" H 1575 1500 50  0000 L CNN
-F 2 "commons_passives_THT:Passive_THT_capacitor_mlcc_W2.54mm_L7.62mm" H 1588 1450 50  0001 C CNN
+F 2 "Capacitor_SMD:C_1206_3216Metric_Pad1.33x1.80mm_HandSolder" H 1588 1450 50  0001 C CNN
 F 3 "~" H 1550 1600 50  0001 C CNN
 	1    1550 1600
