File: subsheet_504.sch (KiCad schematic (older format))
At the start: 35 parts, among them J502 Phono LEFT, J503 Phono RIGHT, U504 LF347N_mu, U508 LMC1992CCN_PHY

Commit message: Resolves #9 : Assign radial THT footprints to polarized capacitors
Parts:
- CP525, CP529, CP535, CP537, CP541, CP543, CP544, CP546, CP547: footprint commons_passives_THT:Passive_THT_capacitor_polarized_W6.35mm_L20.32mm -> Capacitor_THT:C_Radial_D6.3mm_H11.0mm_P2.50mm
- CP542: footprint commons_passives_THT:Passive_THT_capacitor_polarized_W5.08mm_L17.78mm -> Capacitor_THT:C_Radial_D5.0mm_H11.0mm_P2.00mm
Changed lines of the file:
@@
 F 0 "CP535" H 3550 2450 50  0000 L CNN
 F 1 "47uF" H 3550 2250 50  0000 L CNN
-F 2 "commons_passives_THT:Passive_THT_capacitor_polarized_W6.35mm_L20.32mm" H 3500 2350 50  0001 C CNN
+F 2 "Capacitor_THT:C_Radial_D6.3mm_H11.0mm_P2.50mm" H 3500 2350 50  0001 C CNN
 F 3 "~" H 3500 2350 50  0001 C CNN
 	1    3500 2350
@@
 F 0 "CP541" V 1350 950 50  0000 L CNN
 F 1 "47uF" V 1650 950 50  0000 L CNN
-F 2 "commons_passives_THT:Passive_THT_capacitor_polarized_W6.35mm_L20.32mm" H 1500 1050 50  0001 C CNN
+F 2 "Capacitor_THT:C_Radial_D6.3mm_H11.0mm_P2.50mm" H 1500 1050 50  0001 C CNN
 F 3 "~" H 1500 1050 50  0001 C CNN
 	1    1500 1050
@@
 F 0 "CP546" V 1350 1450 50  0000 L CNN
 F 1 "47uF" V 1650 1450 50  0000 L CNN
-F 2 "commons_passives_THT:Passive_THT_capacitor_polarized_W6.35mm_L20.32mm" H 1500 1550 50  0001 C CNN
+F 2 "Capacitor_THT:C_Radial_D6.3mm_H11.0mm_P2.50mm" H 1500 1550 50  0001 C CNN
 F 3 "~" H 1500 1550 50  0001 C CNN
 	1    1500 1550
@@
 F 0 "CP544" V 1350 3450 50  0000 L CNN
 F 1 "47uF" V 1350 3950 50  0000 L CNN
-F 2 "commons_passives_THT:Passive_THT_capacitor_polarized_W6.35mm_L20.32mm" H 1400 3800 50  0001 C CNN
+F 2 "Capacitor_THT:C_Radial_D6.3mm_H11.0mm_P2.50mm" H 1400 3800 50  0001 C CNN
 F 3 "~" H 1400 3800 50  0001 C CNN
 	1    1400 3800
@@
 F 0 "CP547" V 6850 3800 50  0000 L CNN
 F 1 "47uF" V 6850 3450 50  0000 L CNN
-F 2 "commons_passives_THT:Passive_THT_capacitor_polarized_W6.35mm_L20.32mm" H 6800 3700 50  0001 C CNN
+F 2 "Capacitor_THT:C_Radial_D6.3mm_H11.0mm_P2.50mm" H 6800 3700 50  0001 C CNN
 F 3 "~" H 6800 3700 50  0001 C CNN
 	1    6800 3700
@@
 F 0 "CP525" H 1400 6050 50  0000 L CNN
 F 1 "47uF" H 1450 5950 50  0000 L CNN
-F 2 "commons_passives_THT:Passive_THT_capacitor_polarized_W6.35mm_L20.32mm" H 1750 6000 50  0001 C CNN
+F 2 "Capacitor_THT:C_Radial_D6.3mm_H11.0mm_P2.50mm" H 1750 6000 50  0001 C CNN
 F 3 "~" H 1750 6000 50  0001 C CNN
 	1    1750 6000
@@
 F 0 "CP537" H 6600 6050 50  0000 L CNN
 F 1 "47uF" H 6600 5950 50  0000 L CNN
-F 2 "commons_passives_THT:Passive_THT_capacitor_polarized_W6.35mm_L20.32mm" H 6500 6000 50  0001 C CNN
+F 2 "Capacitor_THT:C_Radial_D6.3mm_H11.0mm_P2.50mm" H 6500 6000 50  0001 C CNN
 F 3 "~" H 6500 6000 50  0001 C CNN
 	1    6500 6000
@@
 F 0 "CP529" H 2350 5300 50  0000 L CNN
 F 1 "47uF" H 2350 5200 50  0000 L CNN
-F 2 "commons_passives_THT:Passive_THT_capacitor_polarized_W6.35mm_L20.32mm" H 2250 5250 50  0001 C CNN
+F 2 "Capacitor_THT:C_Radial_D6.3mm_H11.0mm_P2.50mm" H 2250 5250 50  0001 C CNN
 F 3 "~" H 2250 5250 50  0001 C CNN
 	1    2250 5250
@@
 F 0 "CP543" H 6100 5300 50  0000 L CNN
 F 1 "47uF" H 6100 5200 50  0000 L CNN
-F 2 "commons_passives_THT:Passive_THT_capacitor_polarized_W6.35mm_L20.32mm" H 6000 5250 50  0001 C CNN
+F 2 "Capacitor_THT:C_Radial_D6.3mm_H11.0mm_P2.50mm" H 6000 5250 50  0001 C CNN
 F 3 "~" H 6000 5250 50  0001 C CNN
 	1    6000 5250
@@
 F 0 "CP542" V 6150 2850 50  0000 L CNN
 F 1 "10uF" V 6050 2900 50  0000 L CNN
-F 2 "commons_passives_THT:Passive_THT_capacitor_polarized_W5.08mm_L17.78mm" H 6100 3200 50  0001 C CNN
+F 2 "Capacitor_THT:C_Radial_D5.0mm_H11.0mm_P2.00mm" H 6100 3200 50  0001 C CNN
 F 3 "~" H 6100 3200 50  0001 C CNN
 	1    6100 3200
