File: subsheet_103.kicad_sch (KiCad schematic)
At the start: 4 parts, among them J103 Cartridge Port

Commit message: replace symbol Device:CP1 by Device:C_Polarized_US
Parts:
- CP110: symbol Device:CP1 -> Device:C_Polarized_US
Changed lines of the file:
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@@
     (pin "2")
   )
-  (symbol (lib_id "Device:CP1") (at 82.55 59.69 0) (unit 1)
+  (symbol (lib_id "Device:C_Polarized_US") (at 82.55 59.69 0) (unit 1)
     (in_bom yes) (on_board yes)
     (property "Reference" "CP110" (id 0) (at 83.185 57.15 0)
