File: subsheet_104.kicad_sch (KiCad schematic)
At the start: 9 parts, among them U104 LM555_TIMER_PHY, U604 MCP101-D_PHY

Commit message: replace symbol Device:CP1 by Device:C_Polarized_US
Parts:
- CP100, CP102: symbol Device:CP1 -> Device:C_Polarized_US
Changed lines of the file:
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@@
     (pin "2")
   )
-  (symbol (lib_id "Device:CP1") (at 69.85 52.07 0) (unit 1)
+  (symbol (lib_id "Device:C_Polarized_US") (at 69.85 52.07 0) (unit 1)
     (in_bom yes) (on_board yes)
     (property "Reference" "CP100" (id 0) (at 71.12 49.53 0)
@@
     (pin "2")
   )
-  (symbol (lib_id "Device:CP1") (at 165.1 52.07 0) (unit 1)
+  (symbol (lib_id "Device:C_Polarized_US") (at 165.1 52.07 0) (unit 1)
     (in_bom yes) (on_board yes)
     (property "Reference" "CP102" (id 0) (at 166.37 49.53 0)
