File: subsheet_105.kicad_sch (KiCad schematic)
At the start: 22 parts, among them J100 Power

Commit message: replace symbol Device:CP1 by Device:C_Polarized_US
Parts:
- CP107: symbol Device:CP1 -> Device:C_Polarized_US
Changed lines of the file:
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@@
     (pin "6")
   )
-  (symbol (lib_id "Device:CP1") (at 95.25 50.8 0) (unit 1)
+  (symbol (lib_id "Device:C_Polarized_US") (at 95.25 50.8 0) (unit 1)
     (in_bom yes) (on_board yes)
     (property "Reference" "CP107" (id 0) (at 95.885 48.26 0)
