File: subsheet_205.kicad_sch (KiCad schematic)
At the start: 23 parts, among them U204 TL497A_DIP-14_500MA_PEAK_STEP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, U205 TL497A_DIP-14_500MA_PEAK_STEP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

Commit message: replace symbol Device:CP1 by Device:C_Polarized_US
Parts:
- CP202, CP204, CP205, CP215, CP216: symbol Device:CP1 -> Device:C_Polarized_US
Changed lines of the file:
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@@
     (pin "2")
   )
-  (symbol (lib_id "Device:CP1") (at 110.49 102.87 90) (unit 1)
+  (symbol (lib_id "Device:C_Polarized_US") (at 110.49 102.87 90) (unit 1)
     (in_bom yes) (on_board yes)
     (property "Reference" "CP202" (id 0) (at 111.76 106.68 90)
@@
     (pin "2")
   )
-  (symbol (lib_id "Device:CP1") (at 138.43 93.98 0) (unit 1)
+  (symbol (lib_id "Device:C_Polarized_US") (at 138.43 93.98 0) (unit 1)
     (in_bom yes) (on_board yes)
     (property "Reference" "CP204" (id 0) (at 139.065 91.44 0)
@@
     (pin "2")
   )
-  (symbol (lib_id "Device:CP1") (at 138.43 72.39 0) (unit 1)
+  (symbol (lib_id "Device:C_Polarized_US") (at 138.43 72.39 0) (unit 1)
     (in_bom yes) (on_board yes)
     (property "Reference" "CP205" (id 0) (at 139.065 69.85 0)
@@
     (pin "2")
   )
-  (symbol (lib_id "Device:CP1") (at 133.35 158.75 0) (unit 1)
+  (symbol (lib_id "Device:C_Polarized_US") (at 133.35 158.75 0) (unit 1)
     (in_bom yes) (on_board yes)
     (property "Reference" "CP215" (id 0) (at 133.985 156.21 0)
@@
     (pin "2")
   )
-  (symbol (lib_id "Device:CP1") (at 146.05 158.75 0) (unit 1)
+  (symbol (lib_id "Device:C_Polarized_US") (at 146.05 158.75 0) (unit 1)
     (in_bom yes) (on_board yes)
     (property "Reference" "CP216" (id 0) (at 146.685 156.21 0)
