File: subsheet_402.kicad_sch (KiCad schematic)
At the start: 33 parts, among them J400 DIN-13S — Video Port, Q400 MMBT3904, Q401 MMBT3904, Q402 MMBT3904, Q403 MMBT3904, U405 74S257_PHY

Commit message: replace symbol Device:CP1 by Device:C_Polarized_US
Parts:
- CP2101: symbol Device:CP1 -> Device:C_Polarized_US
Changed lines of the file:
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@@
     (pin "2")
   )
-  (symbol (lib_id "Device:CP1") (at 25.4 105.41 0) (unit 1)
+  (symbol (lib_id "Device:C_Polarized_US") (at 25.4 105.41 0) (unit 1)
     (in_bom yes) (on_board yes)
     (property "Reference" "CP2101" (id 0) (at 26.035 102.87 0)
