File: subsheet_502.kicad_sch (KiCad schematic)
At the start: 26 parts, among them U500 74F374_OCTAL_D-TYPE_EDGE-TRIG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, U501 74F374_OCTAL_D-TYPE_EDGE-TRIG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, U502 DAC0802LCN_PHY, U503 DAC0802LCN_PHY

Commit message: replace symbol Device:CP1 by Device:C_Polarized_US
Parts:
- CP558, CP561: symbol Device:CP1 -> Device:C_Polarized_US
Changed lines of the file:
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@@
     (pin "2")
   )
-  (symbol (lib_id "Device:CP1") (at 60.96 44.45 0) (unit 1)
+  (symbol (lib_id "Device:C_Polarized_US") (at 60.96 44.45 0) (unit 1)
     (in_bom yes) (on_board yes)
     (property "Reference" "CP558" (id 0) (at 61.595 41.91 0)
@@
     (pin "2")
   )
-  (symbol (lib_id "Device:CP1") (at 137.16 44.45 0) (unit 1)
+  (symbol (lib_id "Device:C_Polarized_US") (at 137.16 44.45 0) (unit 1)
     (in_bom yes) (on_board yes)
     (property "Reference" "CP561" (id 0) (at 137.795 41.91 0)
