File: subsheet_503.kicad_sch (KiCad schematic)
At the start: 40 parts, among them Q500 UA78L08, U504 LF347N_mu, U505 MF4CN-100_PHY, U506 MF4CN-100_PHY, U507 LF347N_mu

Commit message: replace symbol Device:CP1 by Device:C_Polarized_US
Parts:
- CP508, CP520, CP564, CP566, CP567: symbol Device:CP1 -> Device:C_Polarized_US
Changed lines of the file:
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@@
     (pin "8")
   )
-  (symbol (lib_id "Device:CP1") (at 97.79 49.53 0) (unit 1)
+  (symbol (lib_id "Device:C_Polarized_US") (at 97.79 49.53 0) (unit 1)
     (in_bom yes) (on_board yes)
     (property "Reference" "CP566" (id 0) (at 99.06 46.99 0)
@@
     (pin "8")
   )
-  (symbol (lib_id "Device:CP1") (at 182.88 71.12 0) (unit 1)
+  (symbol (lib_id "Device:C_Polarized_US") (at 182.88 71.12 0) (unit 1)
     (in_bom yes) (on_board yes)
     (property "Reference" "CP567" (id 0) (at 184.15 68.58 0)
@@
     (pin "3")
   )
-  (symbol (lib_id "Device:CP1") (at 139.7 31.75 0) (unit 1)
+  (symbol (lib_id "Device:C_Polarized_US") (at 139.7 31.75 0) (unit 1)
     (in_bom yes) (on_board yes)
     (property "Reference" "CP564" (id 0) (at 140.335 29.21 0)
@@
     (pin "2")
   )
-  (symbol (lib_id "Device:CP1") (at 105.41 163.83 180) (unit 1)
+  (symbol (lib_id "Device:C_Polarized_US") (at 105.41 163.83 180) (unit 1)
     (in_bom yes) (on_board yes)
     (property "Reference" "CP508" (id 0) (at 113.03 162.56 0)
@@
     (pin "2")
   )
-  (symbol (lib_id "Device:CP1") (at 190.5 187.96 180) (unit 1)
+  (symbol (lib_id "Device:C_Polarized_US") (at 190.5 187.96 180) (unit 1)
     (in_bom yes) (on_board yes)
     (property "Reference" "CP520" (id 0) (at 187.96 186.69 0)
