File: subsheet_600.kicad_sch (KiCad schematic)
At the start: 9 parts, among them U600 SIMM_30_PHY, U601 SIMM_30_PHY, U602 SIMM_30_PHY, U603 SIMM_30_PHY

Commit message: replace symbol Device:CP1 by Device:C_Polarized_US
Parts:
- CP600: symbol Device:CP1 -> Device:C_Polarized_US
Changed lines of the file:
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@@
     (pin "2")
   )
-  (symbol (lib_id "Device:CP1") (at 107.95 38.1 0) (unit 1)
+  (symbol (lib_id "Device:C_Polarized_US") (at 107.95 38.1 0) (unit 1)
     (in_bom yes) (on_board yes)
     (property "Reference" "CP600" (id 0) (at 109.22 35.56 0)
@@
   (symbol (lib_id "power:VCC") (at 107.95 29.21 0) (unit 1)
     (in_bom yes) (on_board yes)
-    (property "Reference" "#PWR?" (id 0) (at 107.95 33.02 0)
+    (property "Reference" "#PWR0183" (id 0) (at 107.95 33.02 0)
       (effects (font (size 1.27 1.27)) hide)
     )
@@
   (symbol (lib_id "power:GND") (at 116.84 73.66 0) (unit 1)
     (in_bom yes) (on_board yes)
-    (property "Reference" "#PWR?" (id 0) (at 116.84 80.01 0)
+    (property "Reference" "#PWR0184" (id 0) (at 116.84 80.01 0)
       (effects (font (size 1.27 1.27)) hide)
     )
@@
   (symbol (lib_id "power:VCC") (at 25.4 181.61 0) (unit 1)
     (in_bom yes) (on_board yes)
-    (property "Reference" "#PWR?" (id 0) (at 25.4 185.42 0)
+    (property "Reference" "#PWR0174" (id 0) (at 25.4 185.42 0)
       (effects (font (size 1.27 1.27)) hide)
     )
@@
   (symbol (lib_id "power:GND") (at 38.1 175.26 0) (unit 1)
     (in_bom yes) (on_board yes)
-    (property "Reference" "#PWR?" (id 0) (at 38.1 181.61 0)
+    (property "Reference" "#PWR0173" (id 0) (at 38.1 181.61 0)
       (effects (font (size 1.27 1.27)) hide)
     )
@@
   (symbol (lib_id "power:GND") (at 25.4 199.39 0) (unit 1)
     (in_bom yes) (on_board yes)
-    (property "Reference" "#PWR?" (id 0) (at 25.4 205.74 0)
+    (property "Reference" "#PWR0175" (id 0) (at 25.4 205.74 0)
       (effects (font (size 1.27 1.27)) hide)
     )
@@
   (symbol (lib_id "power:VCC") (at 52.07 228.6 0) (unit 1)
     (in_bom yes) (on_board yes)
-    (property "Reference" "#PWR?" (id 0) (at 52.07 232.41 0)
+    (property "Reference" "#PWR0172" (id 0) (at 52.07 232.41 0)
       (effects (font (size 1.27 1.27)) hide)
     )
@@
   (symbol (lib_id "power:GND") (at 116.84 208.28 0) (unit 1)
     (in_bom yes) (on_board yes)
-    (property "Reference" "#PWR?" (id 0) (at 116.84 214.63 0)
+    (property "Reference" "#PWR0170" (id 0) (at 116.84 214.63 0)
       (effects (font (size 1.27 1.27)) hide)
     )
@@
   (symbol (lib_id "power:VCC") (at 52.07 127 0) (unit 1)
     (in_bom yes) (on_board yes)
-    (property "Reference" "#PWR?" (id 0) (at 52.07 130.81 0)
+    (property "Reference" "#PWR0189" (id 0) (at 52.07 130.81 0)
       (effects (font (size 1.27 1.27)) hide)
     )
@@
   (symbol (lib_id "power:GND") (at 38.1 106.68 0) (unit 1)
     (in_bom yes) (on_board yes)
-    (property "Reference" "#PWR?" (id 0) (at 38.1 113.03 0)
+    (property "Reference" "#PWR0190" (id 0) (at 38.1 113.03 0)
       (effects (font (size 1.27 1.27)) hide)
     )
@@
   (symbol (lib_id "power:GND") (at 177.8 97.79 0) (unit 1)
     (in_bom yes) (on_board yes)
-    (property "Reference" "#PWR?" (id 0) (at 177.8 104.14 0)
+    (property "Reference" "#PWR0179" (id 0) (at 177.8 104.14 0)
       (effects (font (size 1.27 1.27)) hide)
     )
@@
   (symbol (lib_id "power:VCC") (at 52.07 154.94 0) (unit 1)
     (in_bom yes) (on_board yes)
-    (property "Reference" "#PWR?" (id 0) (at 52.07 158.75 0)
+    (property "Reference" "#PWR0171" (id 0) (at 52.07 158.75 0)
       (effects (font (size 1.27 1.27)) hide)
     )
@@
   (symbol (lib_id "power:VCC") (at 130.81 154.94 0) (unit 1)
     (in_bom yes) (on_board yes)
-    (property "Reference" "#PWR?" (id 0) (at 130.81 158.75 0)
+    (property "Reference" "#PWR0168" (id 0) (at 130.81 158.75 0)
       (effects (font (size 1.27 1.27)) hide)
     )
@@
   (symbol (lib_id "power:GND") (at 38.1 208.28 0) (unit 1)
     (in_bom yes) (on_board yes)
-    (property "Reference" "#PWR?" (id 0) (at 38.1 214.63 0)
+    (property "Reference" "#PWR0176" (id 0) (at 38.1 214.63 0)
       (effects (font (size 1.27 1.27)) hide)
     )
@@
   (symbol (lib_id "power:VCC") (at 52.07 53.34 0) (unit 1)
     (in_bom yes) (on_board yes)
-    (property "Reference" "#PWR?" (id 0) (at 52.07 57.15 0)
+    (property "Reference" "#PWR0177" (id 0) (at 52.07 57.15 0)
       (effects (font (size 1.27 1.27)) hide)
     )
@@
   (symbol (lib_id "power:GND") (at 25.4 97.79 0) (unit 1)
     (in_bom yes) (on_board yes)
-    (property "Reference" "#PWR?" (id 0) (at 25.4 104.14 0)
+    (property "Reference" "#PWR0188" (id 0) (at 25.4 104.14 0)
       (effects (font (size 1.27 1.27)) hide)
     )
@@
   (symbol (lib_id "power:GND") (at 38.1 73.66 0) (unit 1)
     (in_bom yes) (on_board yes)
-    (property "Reference" "#PWR?" (id 0) (at 38.1 80.01 0)
+    (property "Reference" "#PWR0186" (id 0) (at 38.1 80.01 0)
       (effects (font (size 1.27 1.27)) hide)
     )
@@
   (symbol (lib_id "power:GND") (at 116.84 175.26 0) (unit 1)
     (in_bom yes) (on_board yes)
-    (property "Reference" "#PWR?" (id 0) (at 116.84 181.61 0)
+    (property "Reference" "#PWR0169" (id 0) (at 116.84 181.61 0)
       (effects (font (size 1.27 1.27)) hide)
     )
@@
   (symbol (lib_id "power:GND") (at 107.95 46.99 0) (unit 1)
     (in_bom yes) (on_board yes)
-    (property "Reference" "#PWR?" (id 0) (at 107.95 53.34 0)
+    (property "Reference" "#PWR0182" (id 0) (at 107.95 53.34 0)
       (effects (font (size 1.27 1.27)) hide)
     )
@@
   (symbol (lib_id "power:GND") (at 116.84 106.68 0) (unit 1)
     (in_bom yes) (on_board yes)
-    (property "Reference" "#PWR?" (id 0) (at 116.84 113.03 0)
+    (property "Reference" "#PWR0180" (id 0) (at 116.84 113.03 0)
       (effects (font (size 1.27 1.27)) hide)
     )
@@
   (symbol (lib_id "power:VCC") (at 130.81 53.34 0) (unit 1)
     (in_bom yes) (on_board yes)
-    (property "Reference" "#PWR?" (id 0) (at 130.81 57.15 0)
+    (property "Reference" "#PWR0185" (id 0) (at 130.81 57.15 0)
       (effects (font (size 1.27 1.27)) hide)
     )
@@
   (symbol (lib_id "power:VCC") (at 130.81 228.6 0) (unit 1)
     (in_bom yes) (on_board yes)
-    (property "Reference" "#PWR?" (id 0) (at 130.81 232.41 0)
+    (property "Reference" "#PWR0167" (id 0) (at 130.81 232.41 0)
       (effects (font (size 1.27 1.27)) hide)
     )
@@
   (symbol (lib_id "power:VCC") (at 25.4 80.01 0) (unit 1)
     (in_bom yes) (on_board yes)
-    (property "Reference" "#PWR?" (id 0) (at 25.4 83.82 0)
+    (property "Reference" "#PWR0187" (id 0) (at 25.4 83.82 0)
       (effects (font (size 1.27 1.27)) hide)
     )
@@
   (symbol (lib_id "power:VCC") (at 177.8 80.01 0) (unit 1)
     (in_bom yes) (on_board yes)
-    (property "Reference" "#PWR?" (id 0) (at 177.8 83.82 0)
+    (property "Reference" "#PWR0178" (id 0) (at 177.8 83.82 0)
       (effects (font (size 1.27 1.27)) hide)
     )
@@
   (symbol (lib_id "power:VCC") (at 130.81 127 0) (unit 1)
     (in_bom yes) (on_board yes)
-    (property "Reference" "#PWR?" (id 0) (at 130.81 130.81 0)
-      (effects (font (size 1.27 1.27)) hide)
-    )
+    (property "Reference" "#PWR0181" (id 0) (at 130.81 130.81 0)
+      (effects (font (size 1.27 1.27)) hide)
+    )
