File: reste-mignon.kicad_pcb (KiCad board)
At the start: 4 copper layers, 0 parts

Commit message: interconnect 68k sockets (dip and plcc)
Parts:
- added C1001: 0.1uF, Capacitor_SMD:C_1206_3216Metric_Pad1.33x1.80mm_HandSolder, F.Cu at (105.6, 531.3)
- added C1002: 1nF, Capacitor_SMD:C_1206_3216Metric_Pad1.33x1.80mm_HandSolder, F.Cu at (105.6, 534.6)
- added C1003: 1nF, Capacitor_SMD:C_1206_3216Metric_Pad1.33x1.80mm_HandSolder, F.Cu at (105.6, 538.0)
- added C101: 0.01uF, Capacitor_SMD:C_1206_3216Metric_Pad1.33x1.80mm_HandSolder, F.Cu at (122.9, 555.5)
- added C104: 0.1uF, Capacitor_SMD:C_1206_3216Metric_Pad1.33x1.80mm_HandSolder, F.Cu at (183.1, 531.0)
- added C105: 0.1uF, Capacitor_SMD:C_1206_3216Metric_Pad1.33x1.80mm_HandSolder, F.Cu at (321.2, 378.1)
- added C106: 0.1uF, Capacitor_SMD:C_1206_3216Metric_Pad1.33x1.80mm_HandSolder, F.Cu at (321.2, 381.4)
- added C108: 0.1uF, Capacitor_SMD:C_1206_3216Metric_Pad1.33x1.80mm_HandSolder, F.Cu at (183.1, 534.4)
- added C109: 0.1uF, Capacitor_SMD:C_1206_3216Metric_Pad1.33x1.80mm_HandSolder, F.Cu at (265.3, 503.0)
- added C111: 0.1uF, Capacitor_SMD:C_1206_3216Metric_Pad1.33x1.80mm_HandSolder, F.Cu at (134.1, 327.7)
- added C112: 0.1uF, Capacitor_SMD:C_1206_3216Metric_Pad1.33x1.80mm_HandSolder, F.Cu at (134.1, 331.1)
- added C113: 0.1uF, Capacitor_SMD:C_1206_3216Metric_Pad1.33x1.80mm_HandSolder, F.Cu at (317.5, 463.1)
- added C114: 0.1uF, Capacitor_SMD:C_1206_3216Metric_Pad1.33x1.80mm_HandSolder, F.Cu at (317.5, 466.5)
- added C1601: 0.1uF, Capacitor_SMD:C_1206_3216Metric_Pad1.33x1.80mm_HandSolder, F.Cu at (184.5, 430.9)
- added C200: 0.1uF, Capacitor_SMD:C_1206_3216Metric_Pad1.33x1.80mm_HandSolder, F.Cu at (314.1, 548.3)
- added C201: 0.1uF, Capacitor_SMD:C_1206_3216Metric_Pad1.33x1.80mm_HandSolder, F.Cu at (314.1, 551.6)
- added C203: 0.1uF, Capacitor_SMD:C_1206_3216Metric_Pad1.33x1.80mm_HandSolder, F.Cu at (198.6, 498.7)
- added C206: 0.1uF, Capacitor_SMD:C_1206_3216Metric_Pad1.33x1.80mm_HandSolder, F.Cu at (198.6, 502.0)
- added C207: 0.1uF, Capacitor_SMD:C_1206_3216Metric_Pad1.33x1.80mm_HandSolder, F.Cu at (322.3, 294.6)
- added C208: 150pF, Capacitor_SMD:C_1206_3216Metric_Pad1.33x1.80mm_HandSolder, F.Cu at (322.3, 298.0)
- added C209: 330pF, Capacitor_SMD:C_1206_3216Metric_Pad1.33x1.80mm_HandSolder, F.Cu at (322.3, 301.4)
- added C210: 0.1uF, Capacitor_SMD:C_1206_3216Metric_Pad1.33x1.80mm_HandSolder, F.Cu at (105.6, 527.9)
- added C2101: 0.1uF, Capacitor_SMD:C_1206_3216Metric_Pad1.33x1.80mm_HandSolder, F.Cu at (88.3, 492.1)
- added C2102: 1uF, Capacitor_SMD:C_1206_3216Metric_Pad1.33x1.80mm_HandSolder, F.Cu at (88.3, 495.4)
- added C214: 0.1uF, Capacitor_SMD:C_1206_3216Metric_Pad1.33x1.80mm_HandSolder, F.Cu at (161.7, 410.7)
- added C217: 0.1uF, Capacitor_SMD:C_1206_3216Metric_Pad1.33x1.80mm_HandSolder, F.Cu at (322.3, 304.7)
- added C218: 270pF, Capacitor_SMD:C_1206_3216Metric_Pad1.33x1.80mm_HandSolder, F.Cu at (322.3, 308.1)
- added C219: 30pF, Capacitor_SMD:C_1206_3216Metric_Pad1.33x1.80mm_HandSolder, F.Cu at (219.1, 364.4)
- added C220: 30pF, Capacitor_SMD:C_1206_3216Metric_Pad1.33x1.80mm_HandSolder, F.Cu at (219.1, 367.8)
- added C221: 0.1uF, Capacitor_SMD:C_1206_3216Metric_Pad1.33x1.80mm_HandSolder, F.Cu at (219.1, 371.1)
- added C222: 100pF, Capacitor_SMD:C_1206_3216Metric_Pad1.33x1.80mm_HandSolder, F.Cu at (198.6, 505.4)
- added C223: 100pF, Capacitor_SMD:C_1206_3216Metric_Pad1.33x1.80mm_HandSolder, F.Cu at (198.6, 508.7)
- added C224: 100pF, Capacitor_SMD:C_1206_3216Metric_Pad1.33x1.80mm_HandSolder, F.Cu at (198.6, 512.1)
- added C225: 100pF, Capacitor_SMD:C_1206_3216Metric_Pad1.33x1.80mm_HandSolder, F.Cu at (198.6, 515.4)
- added C226: 0.1uF, Capacitor_SMD:C_1206_3216Metric_Pad1.33x1.80mm_HandSolder, F.Cu at (218.0, 554.4)
- added C227: 0.1uF, Capacitor_SMD:C_1206_3216Metric_Pad1.33x1.80mm_HandSolder, F.Cu at (314.1, 555.0)
- added C228: 0.1uF, Capacitor_SMD:C_1206_3216Metric_Pad1.33x1.80mm_HandSolder, F.Cu at (198.6, 518.8)
- added C229: 0.1uF, Capacitor_SMD:C_1206_3216Metric_Pad1.33x1.80mm_HandSolder, F.Cu at (219.1, 374.5)
- added C230: 0.1uF, Capacitor_SMD:C_1206_3216Metric_Pad1.33x1.80mm_HandSolder, F.Cu at (219.1, 377.8)
- added C2601: 0.33uF, Capacitor_SMD:C_1206_3216Metric_Pad1.33x1.80mm_HandSolder, F.Cu at (262.0, 304.7)
- added C300: 0.1uF, Capacitor_SMD:C_1206_3216Metric_Pad1.33x1.80mm_HandSolder, F.Cu at (92.0, 557.6)
- added C301: 0.1uF, Capacitor_SMD:C_1206_3216Metric_Pad1.33x1.80mm_HandSolder, F.Cu at (92.0, 560.9)
- added C302: 0.1uF, Capacitor_SMD:C_1206_3216Metric_Pad1.33x1.80mm_HandSolder, F.Cu at (218.0, 557.8)
- added C303: 0.1uF, Capacitor_SMD:C_1206_3216Metric_Pad1.33x1.80mm_HandSolder, F.Cu at (184.5, 420.9)
- added C304: 0.1uF, Capacitor_SMD:C_1206_3216Metric_Pad1.33x1.80mm_HandSolder, F.Cu at (163.8, 520.5)
- added C305: 0.1uF, Capacitor_SMD:C_1206_3216Metric_Pad1.33x1.80mm_HandSolder, F.Cu at (163.8, 523.8)
- added C306: 0.1uF, Capacitor_SMD:C_1206_3216Metric_Pad1.33x1.80mm_HandSolder, F.Cu at (184.5, 424.2)
- added C307: 0.1uF, Capacitor_SMD:C_1206_3216Metric_Pad1.33x1.80mm_HandSolder, F.Cu at (184.5, 427.6)
- added C402: 0.1uF, Capacitor_SMD:C_1206_3216Metric_Pad1.33x1.80mm_HandSolder, F.Cu at (121.1, 422.1)
- added C403: 0.1uF, Capacitor_SMD:C_1206_3216Metric_Pad1.33x1.80mm_HandSolder, F.Cu at (121.1, 425.4)
- added C404: 0.1uF, Capacitor_SMD:C_1206_3216Metric_Pad1.33x1.80mm_HandSolder, F.Cu at (121.1, 428.8)
- added C405: 0.1uF, Capacitor_SMD:C_1206_3216Metric_Pad1.33x1.80mm_HandSolder, F.Cu at (121.1, 432.1)
- added C406: 0.1uF, Capacitor_SMD:C_1206_3216Metric_Pad1.33x1.80mm_HandSolder, F.Cu at (121.1, 435.4)
- added C409: 100pF, Capacitor_SMD:C_1206_3216Metric_Pad1.33x1.80mm_HandSolder, F.Cu at (255.9, 414.2)
- added C411: 0.1uF, Capacitor_SMD:C_1206_3216Metric_Pad1.33x1.80mm_HandSolder, F.Cu at (88.3, 485.4)
- added C412: 0.1uF, Capacitor_SMD:C_1206_3216Metric_Pad1.33x1.80mm_HandSolder, F.Cu at (216.4, 458.9)
- added C413: 0.1uF, Capacitor_SMD:C_1206_3216Metric_Pad1.33x1.80mm_HandSolder, F.Cu at (216.4, 462.3)
- added C414: 0.1uF, Capacitor_SMD:C_1206_3216Metric_Pad1.33x1.80mm_HandSolder, F.Cu at (88.3, 488.7)
- added C500: 0.1uF, Capacitor_SMD:C_1206_3216Metric_Pad1.33x1.80mm_HandSolder, F.Cu at (250.0, 294.6)
- added C501: 0.1uF, Capacitor_SMD:C_1206_3216Metric_Pad1.33x1.80mm_HandSolder, F.Cu at (250.0, 298.0)
- added C502: 0.1uF, Capacitor_SMD:C_1206_3216Metric_Pad1.33x1.80mm_HandSolder, F.Cu at (250.0, 301.4)
- added C503: 0.01uF, Capacitor_SMD:C_1206_3216Metric_Pad1.33x1.80mm_HandSolder, F.Cu at (255.8, 511.1)
- added C504: 0.1uF, Capacitor_SMD:C_1206_3216Metric_Pad1.33x1.80mm_HandSolder, F.Cu at (255.8, 514.4)
- added C505: 0.001uF, Capacitor_SMD:C_1206_3216Metric_Pad1.33x1.80mm_HandSolder, F.Cu at (250.0, 304.7)
- added C506: 0.001uF, Capacitor_SMD:C_1206_3216Metric_Pad1.33x1.80mm_HandSolder, F.Cu at (250.0, 308.1)
- added C507: 0.1uF, Capacitor_SMD:C_1206_3216Metric_Pad1.33x1.80mm_HandSolder, F.Cu at (255.8, 517.8)
- added C509: 0.001uF, Capacitor_SMD:C_1206_3216Metric_Pad1.33x1.80mm_HandSolder, F.Cu at (250.0, 311.4)
- added C510: 0.001uF, Capacitor_SMD:C_1206_3216Metric_Pad1.33x1.80mm_HandSolder, F.Cu at (250.0, 314.8)
- added C511: 0.1uF, Capacitor_SMD:C_1206_3216Metric_Pad1.33x1.80mm_HandSolder, F.Cu at (256.0, 294.6)
- added C512: 0.1uF, Capacitor_SMD:C_1206_3216Metric_Pad1.33x1.80mm_HandSolder, F.Cu at (256.0, 298.0)
- added C513: 0.1uF, Capacitor_SMD:C_1206_3216Metric_Pad1.33x1.80mm_HandSolder, F.Cu at (256.0, 301.4)
- added C514: 0.1uF, Capacitor_SMD:C_1206_3216Metric_Pad1.33x1.80mm_HandSolder, F.Cu at (256.0, 304.7)
- added C515: 0.01uF, Capacitor_SMD:C_1206_3216Metric_Pad1.33x1.80mm_HandSolder, F.Cu at (255.8, 521.1)
- added C516: 0.1uF, Capacitor_SMD:C_1206_3216Metric_Pad1.33x1.80mm_HandSolder, F.Cu at (255.8, 524.5)
- added C517: 0.001uF, Capacitor_SMD:C_1206_3216Metric_Pad1.33x1.80mm_HandSolder, F.Cu at (256.0, 308.1)
- added C518: 0.001uF, Capacitor_SMD:C_1206_3216Metric_Pad1.33x1.80mm_HandSolder, F.Cu at (256.0, 311.4)
- added C519: 0.1uF, Capacitor_SMD:C_1206_3216Metric_Pad1.33x1.80mm_HandSolder, F.Cu at (255.8, 527.8)
- added C521: 0.001uF, Capacitor_SMD:C_1206_3216Metric_Pad1.33x1.80mm_HandSolder, F.Cu at (256.0, 314.8)
- added C522: 0.001uF, Capacitor_SMD:C_1206_3216Metric_Pad1.33x1.80mm_HandSolder, F.Cu at (262.0, 294.6)
- added C523: 0.1uF, Capacitor_SMD:C_1206_3216Metric_Pad1.33x1.80mm_HandSolder, F.Cu at (262.0, 298.0)
- added C524: 0.1uF, Capacitor_SMD:C_1206_3216Metric_Pad1.33x1.80mm_HandSolder, F.Cu at (295.6, 435.2)
- added C526: 800pF, Capacitor_SMD:C_1206_3216Metric_Pad1.33x1.80mm_HandSolder, F.Cu at (288.8, 345.0)
- added C527: 0.01uF, Capacitor_SMD:C_1206_3216Metric_Pad1.33x1.80mm_HandSolder, F.Cu at (288.8, 348.4)
- added C528: 0.0082uF, Capacitor_SMD:C_1206_3216Metric_Pad1.33x1.80mm_HandSolder, F.Cu at (295.6, 438.6)
- added C531: 0.0082uF, Capacitor_SMD:C_1206_3216Metric_Pad1.33x1.80mm_HandSolder, F.Cu at (295.6, 441.9)
- added C532: 800pF, Capacitor_SMD:C_1206_3216Metric_Pad1.33x1.80mm_HandSolder, F.Cu at (288.8, 351.7)
- added C533: 0.01uF, Capacitor_SMD:C_1206_3216Metric_Pad1.33x1.80mm_HandSolder, F.Cu at (288.8, 355.1)
- added C534: 0.0082uF, Capacitor_SMD:C_1206_3216Metric_Pad1.33x1.80mm_HandSolder, F.Cu at (295.6, 445.3)
- added C536: 0.1uF, Capacitor_SMD:C_1206_3216Metric_Pad1.33x1.80mm_HandSolder, F.Cu at (295.6, 448.6)
- added C538: 0.0082uF, Capacitor_SMD:C_1206_3216Metric_Pad1.33x1.80mm_HandSolder, F.Cu at (295.6, 452.0)
- added C539: 800pF, Capacitor_SMD:C_1206_3216Metric_Pad1.33x1.80mm_HandSolder, F.Cu at (288.8, 358.4)
- added C540: 0.01uF, Capacitor_SMD:C_1206_3216Metric_Pad1.33x1.80mm_HandSolder, F.Cu at (288.8, 361.8)
- added C548: 800pF, Capacitor_SMD:C_1206_3216Metric_Pad1.33x1.80mm_HandSolder, F.Cu at (288.8, 365.1)
- added C549: 0.01uF, Capacitor_SMD:C_1206_3216Metric_Pad1.33x1.80mm_HandSolder, F.Cu at (288.8, 368.5)
- added C550: 0.1uF, Capacitor_SMD:C_1206_3216Metric_Pad1.33x1.80mm_HandSolder, F.Cu at (105.3, 406.6)
- added C551: 0.1uF, Capacitor_SMD:C_1206_3216Metric_Pad1.33x1.80mm_HandSolder, F.Cu at (105.3, 410.0)
- added C552: 0.1uF, Capacitor_SMD:C_1206_3216Metric_Pad1.33x1.80mm_HandSolder, F.Cu at (105.3, 413.4)
- added C553: 0.1uF, Capacitor_SMD:C_1206_3216Metric_Pad1.33x1.80mm_HandSolder, F.Cu at (105.3, 416.7)
- added C554: 0.1uF, Capacitor_SMD:C_1206_3216Metric_Pad1.33x1.80mm_HandSolder, F.Cu at (288.8, 371.8)
- added C555: 0.1uF, Capacitor_SMD:C_1206_3216Metric_Pad1.33x1.80mm_HandSolder, F.Cu at (288.8, 375.2)
- added C556: 0.1uF, Capacitor_SMD:C_1206_3216Metric_Pad1.33x1.80mm_HandSolder, F.Cu at (255.8, 531.2)
- added C557: 0.1uF, Capacitor_SMD:C_1206_3216Metric_Pad1.33x1.80mm_HandSolder, F.Cu at (255.8, 534.5)
- added C559: 0.1uF, Capacitor_SMD:C_1206_3216Metric_Pad1.33x1.80mm_HandSolder, F.Cu at (255.8, 537.9)
- added C562: 0.1uF, Capacitor_SMD:C_1206_3216Metric_Pad1.33x1.80mm_HandSolder, F.Cu at (255.8, 541.2)
- added C565: 0.1uF, Capacitor_SMD:C_1206_3216Metric_Pad1.33x1.80mm_HandSolder, F.Cu at (262.0, 301.4)
- added C632: 0.1uF, Capacitor_SMD:C_1206_3216Metric_Pad1.33x1.80mm_HandSolder, F.Cu at (325.6, 409.8)
- added C633: 0.22uF, Capacitor_SMD:C_1206_3216Metric_Pad1.33x1.80mm_HandSolder, F.Cu at (142.5, 329.6)
- added C634: 0.22uF, Capacitor_SMD:C_1206_3216Metric_Pad1.33x1.80mm_HandSolder, F.Cu at (142.5, 333.0)
- added C635: 0.22uF, Capacitor_SMD:C_1206_3216Metric_Pad1.33x1.80mm_HandSolder, F.Cu at (142.5, 336.3)
- added C636: 0.22uF, Capacitor_SMD:C_1206_3216Metric_Pad1.33x1.80mm_HandSolder, F.Cu at (142.5, 339.7)
- added C900: 0.1uF, Capacitor_SMD:C_1206_3216Metric_Pad1.33x1.80mm_HandSolder, F.Cu at (219.1, 381.2)
- added CP100: 47uF, Capacitor_THT:C_Radial_D6.3mm_H11.0mm_P2.50mm, F.Cu at (104.4, 557.3)
- added CP102: 22uF, Capacitor_THT:C_Radial_D5.0mm_H11.0mm_P2.00mm, F.Cu at (122.2, 550.6)
- added CP107: 100uF, Capacitor_THT:C_Radial_D8.0mm_H11.5mm_P3.50mm, F.Cu at (180.7, 564.6)
- added CP110: 100uF, Capacitor_THT:C_Radial_D8.0mm_H11.5mm_P3.50mm, F.Cu at (255.8, 502.6)
- added CP202: 4.7uF, Capacitor_THT:C_Radial_D5.0mm_H11.0mm_P2.00mm, F.Cu at (309.0, 296.2)
- added CP204: 4.7uF, Capacitor_THT:C_Radial_D5.0mm_H11.0mm_P2.00mm, F.Cu at (309.0, 302.8)
- added CP205: 4.7uF, Capacitor_THT:C_Radial_D5.0mm_H11.0mm_P2.00mm, F.Cu at (309.0, 309.4)
- added CP2101: 47uF, Capacitor_THT:C_Radial_D6.3mm_H11.0mm_P2.50mm, F.Cu at (80.1, 495.5)
- added CP215: 4.7uF, Capacitor_THT:C_Radial_D5.0mm_H11.0mm_P2.00mm, F.Cu at (309.0, 315.9)
- added CP216: 470uF, Capacitor_THT:C_Radial_D12.5mm_H20.0mm_P5.00mm, F.Cu at (294.7, 333.1)
- added CP416: 47uF, Capacitor_THT:C_Radial_D6.3mm_H11.0mm_P2.50mm, F.Cu at (80.1, 487.6)
- added CP508: 47uF, Capacitor_THT:C_Radial_D6.3mm_H11.0mm_P2.50mm, F.Cu at (241.8, 296.9)
- added CP520: 47uF, Capacitor_THT:C_Radial_D6.3mm_H11.0mm_P2.50mm, F.Cu at (241.8, 304.8)
- added CP525: 47uF, Capacitor_THT:C_Radial_D6.3mm_H11.0mm_P2.50mm, F.Cu at (271.7, 437.5)
- added CP529: 47uF, Capacitor_THT:C_Radial_D6.3mm_H11.0mm_P2.50mm, F.Cu at (271.7, 445.3)
- added CP535: 47uF, Capacitor_THT:C_Radial_D6.3mm_H11.0mm_P2.50mm, F.Cu at (271.7, 453.2)
- added CP537: 47uF, Capacitor_THT:C_Radial_D6.3mm_H11.0mm_P2.50mm, F.Cu at (279.6, 437.5)
- added CP541: 47uF, Capacitor_THT:C_Radial_D6.3mm_H11.0mm_P2.50mm, F.Cu at (279.6, 445.3)
- added CP542: 10uF, Capacitor_THT:C_Radial_D5.0mm_H11.0mm_P2.00mm, F.Cu at (271.3, 460.4)
- added CP543: 47uF, Capacitor_THT:C_Radial_D6.3mm_H11.0mm_P2.50mm, F.Cu at (279.6, 453.2)
- added CP544: 47uF, Capacitor_THT:C_Radial_D6.3mm_H11.0mm_P2.50mm, F.Cu at (287.4, 437.5)
- added CP546: 47uF, Capacitor_THT:C_Radial_D6.3mm_H11.0mm_P2.50mm, F.Cu at (287.4, 445.3)
- added CP547: 47uF, Capacitor_THT:C_Radial_D6.3mm_H11.0mm_P2.50mm, F.Cu at (287.4, 453.2)
- added CP558: 100uF, Capacitor_THT:C_Radial_D8.0mm_H11.5mm_P3.50mm, F.Cu at (291.0, 541.2)
- added CP561: 100uF, Capacitor_THT:C_Radial_D8.0mm_H11.5mm_P3.50mm, F.Cu at (291.0, 550.7)
- added CP564: 100uF, Capacitor_THT:C_Radial_D8.0mm_H11.5mm_P3.50mm, F.Cu at (268.0, 328.9)
- added CP566: 47uF, Capacitor_THT:C_Radial_D6.3mm_H11.0mm_P2.50mm, F.Cu at (241.8, 312.6)
- added CP567: 47uF, Capacitor_THT:C_Radial_D6.3mm_H11.0mm_P2.50mm, F.Cu at (241.8, 320.4)
- added CP600: 100uF, Capacitor_THT:C_Radial_D8.0mm_H11.5mm_P3.50mm, F.Cu at (148.5, 332.7)
- added D100: 1N914, Diode_SMD:D_SOD-123F, F.Cu at (104.5, 562.9)
- added D200: 1N914, Diode_SMD:D_SOD-123F, F.Cu at (328.0, 294.6)
- added D201: 1N914, Diode_SMD:D_SOD-123F, F.Cu at (328.0, 298.0)
- added D202: 1N914, Diode_SMD:D_SOD-123F, F.Cu at (335.0, 549.7)
- added D203: 1N914, Diode_SMD:D_SOD-123F, F.Cu at (328.0, 301.4)
- added D401: 1N914, Diode_SMD:D_SOD-123F, F.Cu at (285.9, 403.4)
- added D402: 1N914, Diode_SMD:D_SOD-123F, F.Cu at (285.9, 406.7)
- added E0: SolderJumper_2_Open, Jumper:SolderJumper-2_P1.3mm_Open_Pad1.0x1.5mm, F.Cu at (324.8, 387.4)
- added E1: SolderJumper_2_Open, Jumper:SolderJumper-2_P1.3mm_Open_Pad1.0x1.5mm, F.Cu at (324.8, 390.9)
- added E2: SolderJumper_2_Open, Jumper:SolderJumper-2_P1.3mm_Open_Pad1.0x1.5mm, F.Cu at (324.8, 394.5)
- added E3: SolderJumper_2_Open, Jumper:SolderJumper-2_P1.3mm_Open_Pad1.0x1.5mm, F.Cu at (324.8, 398.0)
- added E4: SolderJumper_2_Open, Jumper:SolderJumper-2_P1.3mm_Open_Pad1.0x1.5mm, F.Cu at (324.8, 401.6)
- added E5: SolderJumper_2_Open, Jumper:SolderJumper-2_P1.3mm_Open_Pad1.0x1.5mm, F.Cu at (329.2, 387.4)
- added E6: SolderJumper_2_Open, Jumper:SolderJumper-2_P1.3mm_Open_Pad1.0x1.5mm, F.Cu at (329.2, 390.9)
- added E7: SolderJumper_2_Open, Jumper:SolderJumper-2_P1.3mm_Open_Pad1.0x1.5mm, F.Cu at (329.2, 394.5)
- added FB100: Ferrite Bead, Inductor_SMD:L_1206_3216Metric_Pad1.22x1.90mm_HandSolder, F.Cu at (265.4, 499.6)
- added FB401: Ferrite Bead, Inductor_SMD:L_1206_3216Metric_Pad1.22x1.90mm_HandSolder, F.Cu at (88.3, 498.8)
- added FB402: Ferrite Bead, Inductor_SMD:L_1206_3216Metric_Pad1.22x1.90mm_HandSolder, F.Cu at (88.3, 502.3)
- added FB410: Ferrite Bead, Inductor_SMD:L_1206_3216Metric_Pad1.22x1.90mm_HandSolder, F.Cu at (280.2, 400.0)
- added FB500: Ferrite Bead, Inductor_SMD:L_1206_3216Metric_Pad1.22x1.90mm_HandSolder, F.Cu at (300.8, 345.1)
- added FB501: Ferrite Bead, Inductor_SMD:L_1206_3216Metric_Pad1.22x1.90mm_HandSolder, F.Cu at (300.8, 348.5)
- added FB502: Ferrite Bead, Inductor_SMD:L_1206_3216Metric_Pad1.22x1.90mm_HandSolder, F.Cu at (300.8, 352.0)
- added FB503: Ferrite Bead, Inductor_SMD:L_1206_3216Metric_Pad1.22x1.90mm_HandSolder, F.Cu at (300.8, 355.4)
- added FB508: Ferrite Bead, Inductor_SMD:L_1206_3216Metric_Pad1.22x1.90mm_HandSolder, F.Cu at (300.8, 358.9)
- added H2001: M2.5, mounting-holes:MountingHole_2.7mm_M2.5_clear_10mm, F.Cu at (237.1, 422.7)
- added H2002: M2.5, mounting-holes:MountingHole_2.7mm_M2.5_clear_10mm, F.Cu at (237.1, 429.6)
- added H2003: M2.5, mounting-holes:MountingHole_2.7mm_M2.5_clear_10mm, F.Cu at (237.1, 436.6)
- added H2004: M2.5, mounting-holes:MountingHole_2.7mm_M2.5_clear_10mm, F.Cu at (237.1, 443.5)
- added H701: UNC 6-32, unc-mounting-holes:MountingHole_3.7mm_UTS_6_Pad_Via, F.Cu at (144.6, 534.4)
- added H702: UNC 6-32, unc-mounting-holes:MountingHole_3.7mm_UTS_6_Pad_Via, F.Cu at (144.6, 544.6)
- added H703: UNC 6-32, unc-mounting-holes:MountingHole_3.7mm_UTS_6_Pad_Via, F.Cu at (144.6, 554.7)
- added H704: UNC 6-32, unc-mounting-holes:MountingHole_3.7mm_UTS_6_Pad_Via, F.Cu at (154.7, 534.4)
- added H705: UNC 6-32, unc-mounting-holes:MountingHole_3.7mm_UTS_6_Pad_Via, F.Cu at (154.7, 544.6)
- added H706: UNC 6-32, unc-mounting-holes:MountingHole_3.7mm_UTS_6_Pad_Via, F.Cu at (154.7, 554.7)
- added H707: UNC 6-32, unc-mounting-holes:MountingHole_3.7mm_UTS_6_Pad_Via, F.Cu at (164.9, 534.4)
- added H708: UNC 6-32, unc-mounting-holes:MountingHole_3.7mm_UTS_6_Pad_Via, F.Cu at (164.9, 544.6)
- added H709: UNC 6-32, unc-mounting-holes:MountingHole_3.7mm_UTS_6_Pad_Via, F.Cu at (164.9, 554.7)
- added H710: UNC 6-32, unc-mounting-holes:MountingHole_3.7mm_UTS_6_Pad_Via, F.Cu at (175.0, 534.4)
- added H711: UNC 6-32, unc-mounting-holes:MountingHole_3.7mm_UTS_6_Pad_Via, F.Cu at (175.0, 544.6)
- added H712: UNC 6-32, unc-mounting-holes:MountingHole_3.7mm_UTS_6_Pad_Via, F.Cu at (175.0, 554.7)
- added H713: M2.5, mounting-holes:MountingHole_2.7mm_M2.5_clear_10mm, F.Cu at (143.0, 563.3)
- added H714: M2.5, mounting-holes:MountingHole_2.7mm_M2.5_clear_10mm, F.Cu at (143.0, 570.2)
- added H715: M2.5, mounting-holes:MountingHole_2.7mm_M2.5_clear_10mm, F.Cu at (149.9, 563.3)
- added H716: M2.5, mounting-holes:MountingHole_2.7mm_M2.5_clear_10mm, F.Cu at (149.9, 570.2)
- added H717: M2.5, mounting-holes:MountingHole_2.7mm_M2.5_clear_10mm, F.Cu at (156.9, 563.3)
- added H718: M2.5, mounting-holes:MountingHole_2.7mm_M2.5_clear_10mm, F.Cu at (156.9, 570.2)
- added J100: Power, Connector_Molex:Molex_KK-254_AE-6410-06A_1x06_P2.54mm_Vertical, F.Cu at (162.6, 563.7)
- added J1001: RJ11S - To Mega ST(e)/TT Keyboard, Connector_RJ:RJ12_Amphenol_54601, F.Cu at (107.2, 508.4)
- added J103: Cartridge Port, atari-interconnect:socket-edge-pcb_40p_P2.01mm, F.Cu at (288.1, 480.3)
- added J1101: Parallel and Serial breakout, Connector_PinHeader_2.54mm:PinHeader_2x14_P2.54mm_Vertical, F.Cu at (161.1, 367.1)
- added J1601: Like MegaSTE J402, Connector_PinHeader_2.54mm:PinHeader_2x15_P2.54mm_Vertical, F.Cu at (141.8, 421.5)
- added J1701: Jumpers, Connector_PinHeader_2.54mm:PinHeader_2x02_P2.54mm_Vertical, F.Cu at (163.1, 513.9)
- added J1901: ROM[0..6] Breakout, Connector_PinSocket_2.54mm:PinSocket_2x07_P2.54mm_Vertical, F.Cu at (115.8, 422.7)
- added J200: DIN-5S — MIDI OUT/THRU, commons-interconnect_THT:socket-din-5, F.Cu at (310.0, 521.2)
- added J2001: For RGB2HDMI, Connector_PinHeader_2.54mm:PinHeader_2x10_P2.54mm_Vertical, F.Cu at (242.9, 421.5)
- added J201: DIN-5S — MIDI IN, commons-interconnect_THT:socket-din-5, F.Cu at (310.0, 539.8)
- added J202: BRS — To IKBD, atari-interconnect:PinHeader_1x08_P2.54mm_Vertical_Ikbd, F.Cu at (99.7, 508.5)
- added J203: DB-25S Parallel port, commons-interconnect_THT:DSUB-25_Female_Horizontal_P2.77x2.84mm_EdgePinOffset7.70mm_Housed_MountingHolesOffset9.12mm, F.Cu at (183.7, 346.6)
- added J204: DB-25P Serial Port RS-232, commons-interconnect_THT:DSUB-25_Male_Horizontal_P2.77x2.84mm_EdgePinOffset7.70mm_Housed_MountingHolesOffset9.12mm, F.Cu at (206.6, 479.0)
- added J301: DB-19S ACSI Port, atari-interconnect:DSUB-19_Female_Horizontal_P2.77x2.84mm_EdgePinOffset7.70mm_Housed_MountingHolesOffset9.12mm, F.Cu at (182.6, 449.5)
- added J302: Internal FDD Power, Connector_Molex:Molex_KK-254_AE-6410-04A_1x04_P2.54mm_Vertical, F.Cu at (173.0, 522.7)
- added J303: Internal FDD Port, Connector_IDC:IDC-Header_2x17_P2.54mm_Vertical, F.Cu at (144.7, 480.6)
- added J304: DIN-14S — External FDD Port, atari-interconnect:socket-din-14, F.Cu at (182.0, 487.0)
- added J305: No Blitter, Connector_PinHeader_2.54mm:PinHeader_2x02_P2.54mm_Vertical, F.Cu at (313.4, 378.7)
- added J400: DIN-13S — Video Port, atari-interconnect:socket-din-13, F.Cu at (105.3, 495.6)
- added J500: DM-15S — JOY0, commons-interconnect_THT:DSUB-15-HD_Female_Horizontal_P2.29x1.98mm_EdgePinOffset8.35mm_Housed_MountingHolesOffset10.89mm, F.Cu at (273.7, 346.4)
- added J501: DM-15S — JOY1, commons-interconnect_THT:DSUB-15-HD_Female_Horizontal_P2.29x1.98mm_EdgePinOffset8.35mm_Housed_MountingHolesOffset10.89mm, F.Cu at (273.7, 369.3)
- added J502: Phono LEFT, atari-interconnect:socket-rca-5-pins, F.Cu at (275.4, 431.0)
- added J503: Phono RIGHT, atari-interconnect:socket-rca-5-pins, F.Cu at (288.2, 431.0)
- added L203: 220uH, commons_passives_THT:L_Radial_D15.0mm_P5.00mm, F.Cu at (296.0, 301.2)
- added L208: 220uH, commons_passives_THT:L_Radial_D15.0mm_P5.00mm, F.Cu at (296.0, 317.8)
- added Q400: MMBT3904, Package_TO_SOT_SMD:SOT-23, F.Cu at (109.3, 462.9)
- added Q401: MMBT3904, Package_TO_SOT_SMD:SOT-23, F.Cu at (109.3, 467.4)
- added Q402: MMBT3904, Package_TO_SOT_SMD:SOT-23, F.Cu at (109.3, 471.8)
- added Q403: MMBT3904, Package_TO_SOT_SMD:SOT-23, F.Cu at (109.3, 476.2)
- added Q405: MMBT3904, Package_TO_SOT_SMD:SOT-23, F.Cu at (285.5, 410.6)
- added Q500: UA78L08, Package_TO_SOT_THT:TO-92L_Inline_Wide, F.Cu at (276.1, 327.4)
- added R100: 10K, Resistor_SMD:R_1206_3216Metric_Pad1.30x1.75mm_HandSolder, F.Cu at (122.9, 558.8)
- added R101: 12K, Resistor_SMD:R_1206_3216Metric_Pad1.30x1.75mm_HandSolder, F.Cu at (122.9, 562.1)
- added R102: 1K, Resistor_SMD:R_1206_3216Metric_Pad1.30x1.75mm_HandSolder, F.Cu at (128.2, 327.7)
- added R106: 4K7, Resistor_SMD:R_1206_3216Metric_Pad1.30x1.75mm_HandSolder, F.Cu at (327.2, 378.0)
- added R107: 1K, Resistor_SMD:R_1206_3216Metric_Pad1.30x1.75mm_HandSolder, F.Cu at (128.2, 331.0)
- added R109: 2K2, Resistor_SMD:R_1206_3216Metric_Pad1.30x1.75mm_HandSolder, F.Cu at (128.2, 334.2)
- added R110: 2K2, Resistor_SMD:R_1206_3216Metric_Pad1.30x1.75mm_HandSolder, F.Cu at (128.2, 337.5)
- added R1701: 1K, Resistor_SMD:R_1206_3216Metric_Pad1.30x1.75mm_HandSolder, F.Cu at (185.3, 502.8)
- added R203: 5.1, Resistor_SMD:R_1206_3216Metric_Pad1.30x1.75mm_HandSolder, F.Cu at (316.3, 294.6)
- added R206: 12K, Resistor_SMD:R_1206_3216Metric_Pad1.30x1.75mm_HandSolder, F.Cu at (316.3, 297.9)
- added R207: 220, Resistor_SMD:R_1206_3216Metric_Pad1.30x1.75mm_HandSolder, F.Cu at (335.2, 543.1)
- added R208: 1K2, Resistor_SMD:R_1206_3216Metric_Pad1.30x1.75mm_HandSolder, F.Cu at (316.3, 301.2)
- added R209: 1K, Resistor_SMD:R_1206_3216Metric_Pad1.30x1.75mm_HandSolder, F.Cu at (335.2, 546.4)
- added R210: 10K, Resistor_SMD:R_1206_3216Metric_Pad1.30x1.75mm_HandSolder, F.Cu at (111.6, 527.9)
- added R211: 1, Resistor_SMD:R_1206_3216Metric_Pad1.30x1.75mm_HandSolder, F.Cu at (316.3, 304.5)
- added R212: 3K3, Resistor_SMD:R_1206_3216Metric_Pad1.30x1.75mm_HandSolder, F.Cu at (161.7, 404.1)
- added R213: 1K2, Resistor_SMD:R_1206_3216Metric_Pad1.30x1.75mm_HandSolder, F.Cu at (316.3, 307.8)
- added R214: 3K9, Resistor_SMD:R_1206_3216Metric_Pad1.30x1.75mm_HandSolder, F.Cu at (316.3, 311.1)
- added R215: 4K7, Resistor_SMD:R_1206_3216Metric_Pad1.30x1.75mm_HandSolder, F.Cu at (239.2, 364.4)
- added R216: 4K7, Resistor_SMD:R_1206_3216Metric_Pad1.30x1.75mm_HandSolder, F.Cu at (239.2, 367.7)
- added R217: 4K7, Resistor_SMD:R_1206_3216Metric_Pad1.30x1.75mm_HandSolder, F.Cu at (239.2, 371.0)
- added R220: 1K, Resistor_SMD:R_1206_3216Metric_Pad1.30x1.75mm_HandSolder, F.Cu at (161.7, 407.4)
- added R2701: 10K, Resistor_SMD:R_1206_3216Metric_Pad1.30x1.75mm_HandSolder, F.Cu at (264.6, 471.2)
- added R302: 1K, Resistor_SMD:R_1206_3216Metric_Pad1.30x1.75mm_HandSolder, F.Cu at (185.3, 496.2)
- added R303: 1K, Resistor_SMD:R_1206_3216Metric_Pad1.30x1.75mm_HandSolder, F.Cu at (217.9, 561.1)
- added R307: 220, Resistor_SMD:R_1206_3216Metric_Pad1.30x1.75mm_HandSolder, F.Cu at (185.3, 499.5)
- added R406: 1K, Resistor_SMD:R_1206_3216Metric_Pad1.30x1.75mm_HandSolder, F.Cu at (80.4, 462.3)
- added R407: 75, Resistor_SMD:R_1206_3216Metric_Pad1.30x1.75mm_HandSolder, F.Cu at (80.4, 465.6)
- added R408: 2K, Resistor_SMD:R_1206_3216Metric_Pad1.30x1.75mm_HandSolder, F.Cu at (80.4, 468.9)
- added R409: 150, Resistor_SMD:R_1206_3216Metric_Pad1.30x1.75mm_HandSolder, F.Cu at (80.4, 472.2)
- added R411: 12K, Resistor_SMD:R_1206_3216Metric_Pad1.30x1.75mm_HandSolder, F.Cu at (198.6, 458.9)
- added R412: 1K5, Resistor_SMD:R_1206_3216Metric_Pad1.30x1.75mm_HandSolder, F.Cu at (198.6, 462.2)
- added R413: 1K, Resistor_SMD:R_1206_3216Metric_Pad1.30x1.75mm_HandSolder, F.Cu at (80.4, 475.5)
- added R414: 3K, Resistor_SMD:R_1206_3216Metric_Pad1.30x1.75mm_HandSolder, F.Cu at (198.6, 465.5)
- added R415: 6K2, Resistor_SMD:R_1206_3216Metric_Pad1.30x1.75mm_HandSolder, F.Cu at (198.6, 468.8)
- added R416: 12K, Resistor_SMD:R_1206_3216Metric_Pad1.30x1.75mm_HandSolder, F.Cu at (198.6, 472.1)
- added R417: 1K5, Resistor_SMD:R_1206_3216Metric_Pad1.30x1.75mm_HandSolder, F.Cu at (204.5, 458.9)
- added R418: 3K, Resistor_SMD:R_1206_3216Metric_Pad1.30x1.75mm_HandSolder, F.Cu at (204.5, 462.2)
- added R419: 6K2, Resistor_SMD:R_1206_3216Metric_Pad1.30x1.75mm_HandSolder, F.Cu at (204.5, 465.5)
- added R420: 75, Resistor_SMD:R_1206_3216Metric_Pad1.30x1.75mm_HandSolder, F.Cu at (80.4, 478.8)
- added R421: 1K, Resistor_SMD:R_1206_3216Metric_Pad1.30x1.75mm_HandSolder, F.Cu at (114.0, 441.9)
- added R422: 12K, Resistor_SMD:R_1206_3216Metric_Pad1.30x1.75mm_HandSolder, F.Cu at (204.5, 468.8)
- added R423: 2K, Resistor_SMD:R_1206_3216Metric_Pad1.30x1.75mm_HandSolder, F.Cu at (80.4, 482.1)
- added R424: 1K5, Resistor_SMD:R_1206_3216Metric_Pad1.30x1.75mm_HandSolder, F.Cu at (204.5, 472.1)
- added R425: 150, Resistor_SMD:R_1206_3216Metric_Pad1.30x1.75mm_HandSolder, F.Cu at (86.4, 462.3)
- added R426: 3K, Resistor_SMD:R_1206_3216Metric_Pad1.30x1.75mm_HandSolder, F.Cu at (210.4, 458.9)
- added R428: 6K2, Resistor_SMD:R_1206_3216Metric_Pad1.30x1.75mm_HandSolder, F.Cu at (210.4, 462.2)
- added R429: 1K, Resistor_SMD:R_1206_3216Metric_Pad1.30x1.75mm_HandSolder, F.Cu at (86.4, 465.6)
- added R430: 1K, Resistor_SMD:R_1206_3216Metric_Pad1.30x1.75mm_HandSolder, F.Cu at (210.4, 465.5)
- added R431: 1K2, Resistor_SMD:R_1206_3216Metric_Pad1.30x1.75mm_HandSolder, F.Cu at (86.4, 468.9)
- added R432: 75, Resistor_SMD:R_1206_3216Metric_Pad1.30x1.75mm_HandSolder, F.Cu at (86.4, 472.2)
- added R433: 2K, Resistor_SMD:R_1206_3216Metric_Pad1.30x1.75mm_HandSolder, F.Cu at (86.4, 475.5)
- added R434: 150, Resistor_SMD:R_1206_3216Metric_Pad1.30x1.75mm_HandSolder, F.Cu at (86.4, 478.8)
- added R435: 33, Resistor_SMD:R_1206_3216Metric_Pad1.30x1.75mm_HandSolder, F.Cu at (86.4, 482.1)
- added R437: 33, Resistor_SMD:R_1206_3216Metric_Pad1.30x1.75mm_HandSolder, F.Cu at (92.3, 462.3)
- added R438: 27, Resistor_SMD:R_1206_3216Metric_Pad1.30x1.75mm_HandSolder, F.Cu at (92.3, 465.6)
- added R440: 1K, Resistor_SMD:R_1206_3216Metric_Pad1.30x1.75mm_HandSolder, F.Cu at (92.3, 468.9)
- added R441: 100, Resistor_SMD:R_1206_3216Metric_Pad1.30x1.75mm_HandSolder, F.Cu at (92.3, 472.2)
- added R472: 4K7, Resistor_SMD:R_1206_3216Metric_Pad1.30x1.75mm_HandSolder, F.Cu at (92.3, 475.5)
- added R473: 10K, Resistor_SMD:R_1206_3216Metric_Pad1.30x1.75mm_HandSolder, F.Cu at (280.1, 403.3)
- added R474: 100, Resistor_SMD:R_1206_3216Metric_Pad1.30x1.75mm_HandSolder, F.Cu at (280.1, 406.6)
- added R475: 150, Resistor_SMD:R_1206_3216Metric_Pad1.30x1.75mm_HandSolder, F.Cu at (280.1, 409.9)
- added R500: 8K2 1%, Resistor_SMD:R_1206_3216Metric_Pad1.30x1.75mm_HandSolder, F.Cu at (261.8, 511.0)
- added R501: 10K 1%, Resistor_SMD:R_1206_3216Metric_Pad1.30x1.75mm_HandSolder, F.Cu at (249.9, 318.1)
- added R502: 10K 1%, Resistor_SMD:R_1206_3216Metric_Pad1.30x1.75mm_HandSolder, F.Cu at (249.9, 321.4)
- added R503: 10K 1%, Resistor_SMD:R_1206_3216Metric_Pad1.30x1.75mm_HandSolder, F.Cu at (249.9, 324.6)
- added R504: 10K 1%, Resistor_SMD:R_1206_3216Metric_Pad1.30x1.75mm_HandSolder, F.Cu at (249.9, 327.9)
- added R505: 10K, Resistor_SMD:R_1206_3216Metric_Pad1.30x1.75mm_HandSolder, F.Cu at (261.8, 514.3)
- added R506: 10K 1%, Resistor_SMD:R_1206_3216Metric_Pad1.30x1.75mm_HandSolder, F.Cu at (261.8, 517.6)
- added R507: 1K8 1%, Resistor_SMD:R_1206_3216Metric_Pad1.30x1.75mm_HandSolder, F.Cu at (255.9, 318.1)
- added R508: 8K2 1%, Resistor_SMD:R_1206_3216Metric_Pad1.30x1.75mm_HandSolder, F.Cu at (261.8, 520.9)
- added R509: 8K2 1%, Resistor_SMD:R_1206_3216Metric_Pad1.30x1.75mm_HandSolder, F.Cu at (261.8, 524.2)
- added R510: 10K 1%, Resistor_SMD:R_1206_3216Metric_Pad1.30x1.75mm_HandSolder, F.Cu at (255.9, 321.4)
- added R511: 10K 1%, Resistor_SMD:R_1206_3216Metric_Pad1.30x1.75mm_HandSolder, F.Cu at (255.9, 324.6)
- added R512: 10K 1%, Resistor_SMD:R_1206_3216Metric_Pad1.30x1.75mm_HandSolder, F.Cu at (255.9, 327.9)
- added R513: 10K 1%, Resistor_SMD:R_1206_3216Metric_Pad1.30x1.75mm_HandSolder, F.Cu at (261.9, 318.1)
- added R514: 10K, Resistor_SMD:R_1206_3216Metric_Pad1.30x1.75mm_HandSolder, F.Cu at (261.8, 527.5)
- added R515: 10K 1%, Resistor_SMD:R_1206_3216Metric_Pad1.30x1.75mm_HandSolder, F.Cu at (261.8, 530.8)
- added R516: 1K8 1%, Resistor_SMD:R_1206_3216Metric_Pad1.30x1.75mm_HandSolder, F.Cu at (261.9, 321.4)
- added R517: 8K2 1%, Resistor_SMD:R_1206_3216Metric_Pad1.30x1.75mm_HandSolder, F.Cu at (261.8, 534.1)
- added R518: 1M, Resistor_SMD:R_1206_3216Metric_Pad1.30x1.75mm_HandSolder, F.Cu at (294.8, 345.0)
- added R519: 470, Resistor_SMD:R_1206_3216Metric_Pad1.30x1.75mm_HandSolder, F.Cu at (294.8, 348.3)
- added R520: 1K, Resistor_SMD:R_1206_3216Metric_Pad1.30x1.75mm_HandSolder, F.Cu at (252.8, 458.0)
- added R521: 1M, Resistor_SMD:R_1206_3216Metric_Pad1.30x1.75mm_HandSolder, F.Cu at (294.8, 351.6)
- added R523: 470, Resistor_SMD:R_1206_3216Metric_Pad1.30x1.75mm_HandSolder, F.Cu at (294.8, 354.9)
- added R524: 3K6, Resistor_SMD:R_1206_3216Metric_Pad1.30x1.75mm_HandSolder, F.Cu at (252.8, 461.3)
- added R525: 10K, Resistor_SMD:R_1206_3216Metric_Pad1.30x1.75mm_HandSolder, F.Cu at (252.8, 464.6)
- added R527: 10K, Resistor_SMD:R_1206_3216Metric_Pad1.30x1.75mm_HandSolder, F.Cu at (252.8, 467.9)
- added R528: 1M, Resistor_SMD:R_1206_3216Metric_Pad1.30x1.75mm_HandSolder, F.Cu at (294.8, 358.1)
- added R529: 470, Resistor_SMD:R_1206_3216Metric_Pad1.30x1.75mm_HandSolder, F.Cu at (294.8, 361.4)
- added R530: 10K, Resistor_SMD:R_1206_3216Metric_Pad1.30x1.75mm_HandSolder, F.Cu at (252.8, 471.2)
- added R531: 51K, Resistor_SMD:R_1206_3216Metric_Pad1.30x1.75mm_HandSolder, F.Cu at (258.7, 458.0)
- added R533: 1K, Resistor_SMD:R_1206_3216Metric_Pad1.30x1.75mm_HandSolder, F.Cu at (258.7, 461.3)
- added R535: 1M, Resistor_SMD:R_1206_3216Metric_Pad1.30x1.75mm_HandSolder, F.Cu at (294.8, 364.7)
- added R536: 470, Resistor_SMD:R_1206_3216Metric_Pad1.30x1.75mm_HandSolder, F.Cu at (294.8, 368.0)
- added R537: 3K6, Resistor_SMD:R_1206_3216Metric_Pad1.30x1.75mm_HandSolder, F.Cu at (258.7, 464.6)
- added R538: 10K, Resistor_SMD:R_1206_3216Metric_Pad1.30x1.75mm_HandSolder, F.Cu at (258.7, 467.9)
- added R539: 51K, Resistor_SMD:R_1206_3216Metric_Pad1.30x1.75mm_HandSolder, F.Cu at (258.7, 471.2)
- added R540: 1K, Resistor_SMD:R_1206_3216Metric_Pad1.30x1.75mm_HandSolder, F.Cu at (264.6, 458.0)
- added R541: 1K, Resistor_SMD:R_1206_3216Metric_Pad1.30x1.75mm_HandSolder, F.Cu at (264.6, 461.3)
- added R542: 10, Resistor_SMD:R_1206_3216Metric_Pad1.30x1.75mm_HandSolder, F.Cu at (261.8, 537.4)
- added R543: 10, Resistor_SMD:R_1206_3216Metric_Pad1.30x1.75mm_HandSolder, F.Cu at (261.8, 540.6)
- added R545: 100K 1%, Resistor_SMD:R_1206_3216Metric_Pad1.30x1.75mm_HandSolder, F.Cu at (261.9, 324.6)
- added R546: 100K 1%, Resistor_SMD:R_1206_3216Metric_Pad1.30x1.75mm_HandSolder, F.Cu at (261.9, 327.9)
- added R590: 270K, Resistor_SMD:R_1206_3216Metric_Pad1.30x1.75mm_HandSolder, F.Cu at (264.6, 464.6)
- added R591: 270K, Resistor_SMD:R_1206_3216Metric_Pad1.30x1.75mm_HandSolder, F.Cu at (264.6, 467.9)
- added RN1501: 10K ×4, Resistor_SMD:R_Array_Convex_4x0603, F.Cu at (217.1, 550.4)
- added RN1502: 10K ×4, Resistor_SMD:R_Array_Convex_4x0603, F.Cu at (221.2, 550.4)
- added RN1601: 68 ×4, Resistor_SMD:R_Array_Convex_4x0603, F.Cu at (148.8, 470.1)
- added RN1602: 68 ×4, Resistor_SMD:R_Array_Convex_4x0603, F.Cu at (152.9, 470.1)
- added RN1603: 68 ×4, Resistor_SMD:R_Array_Convex_4x0603, F.Cu at (157.1, 470.1)
- added RN1701: 1K ×4, Resistor_SMD:R_Array_Convex_4x0603, F.Cu at (172.8, 516.3)
- added RN1702: 1K ×4, Resistor_SMD:R_Array_Convex_4x0603, F.Cu at (176.9, 516.3)
- added RN1703: 47 ×4, Resistor_SMD:R_Array_Convex_4x0603, F.Cu at (181.1, 516.3)
- added RN1704: 1K ×4, Resistor_SMD:R_Array_Convex_4x0603, F.Cu at (185.2, 516.3)
- added RN1901: 33 ×4, Resistor_SMD:R_Array_Convex_4x0603, F.Cu at (79.5, 456.3)
- added RN1902: 33 ×4, Resistor_SMD:R_Array_Convex_4x0603, F.Cu at (83.7, 456.3)
- added RN1903: 68 ×4, Resistor_SMD:R_Array_Convex_4x0603, F.Cu at (87.8, 456.3)
- added RN1904: 68 ×4, Resistor_SMD:R_Array_Convex_4x0603, F.Cu at (92.0, 456.3)
- added RN1905: 68 ×4, Resistor_SMD:R_Array_Convex_4x0603, F.Cu at (96.1, 456.3)
- added RN201: 1K2 ×4, Resistor_SMD:R_Array_Convex_4x0603, F.Cu at (106.5, 328.4)
- added RN202: 1K2 ×4, Resistor_SMD:R_Array_Convex_4x0603, F.Cu at (110.7, 328.4)
- added RN203: 2K2 ×4, Resistor_SMD:R_Array_Convex_4x0603, F.Cu at (114.8, 328.4)
- added RN204: 2K2 ×4, Resistor_SMD:R_Array_Convex_4x0603, F.Cu at (119.0, 328.4)
- added RN205: 2K2 ×4, Resistor_SMD:R_Array_Convex_4x0603, F.Cu at (123.1, 328.4)
- added RN206: 2K2 ×4, Resistor_SMD:R_Array_Convex_4x0603, F.Cu at (106.5, 333.1)
- added RN207: 2K2 ×4, Resistor_SMD:R_Array_Convex_4x0603, F.Cu at (110.7, 333.1)
- added RN208: 2K2 ×4, Resistor_SMD:R_Array_Convex_4x0603, F.Cu at (114.8, 333.1)
- added RN209: 2K2 ×4, Resistor_SMD:R_Array_Convex_4x0603, F.Cu at (119.0, 333.1)
- added RN210: 2K2 ×4, Resistor_SMD:R_Array_Convex_4x0603, F.Cu at (123.1, 333.1)
- added RN211: 2K2 ×4, Resistor_SMD:R_Array_Convex_4x0603, F.Cu at (106.5, 337.9)
- added RN212: 2K2 ×4, Resistor_SMD:R_Array_Convex_4x0603, F.Cu at (110.7, 337.9)
- added RN213: 2K2 ×4, Resistor_SMD:R_Array_Convex_4x0603, F.Cu at (114.8, 337.9)
- added RN2401: 4K7 ×4, Resistor_SMD:R_Array_Convex_4x0603, F.Cu at (79.5, 407.4)
- added RN2402: 4K7 ×4, Resistor_SMD:R_Array_Convex_4x0603, F.Cu at (83.7, 407.4)
- added RN2403: 4K7 ×4, Resistor_SMD:R_Array_Convex_4x0603, F.Cu at (87.8, 407.4)
- added RN2404: 4K7 ×4, Resistor_SMD:R_Array_Convex_4x0603, F.Cu at (92.0, 407.4)
- added RN2405: 4K7 ×4, Resistor_SMD:R_Array_Convex_4x0603, F.Cu at (96.1, 407.4)
- added RN2406: 4K7 ×4, Resistor_SMD:R_Array_Convex_4x0603, F.Cu at (100.3, 407.4)
- added RN2901: 10K ×4, Resistor_SMD:R_Array_Convex_4x0603, F.Cu at (324.7, 405.7)
- added RN2902: 10K ×4, Resistor_SMD:R_Array_Convex_4x0603, F.Cu at (328.9, 405.7)
- added RN901: 4K7 ×4, Resistor_SMD:R_Array_Convex_4x0603, F.Cu at (301.6, 558.2)
- added RN902: 220 ×4, Resistor_SMD:R_Array_Convex_4x0603, F.Cu at (305.7, 558.2)
- added S100: RESET switch, atari-interconnect:switch-spdt-momentary-action_Reset_pushbutton, F.Cu at (117.1, 555.0)
- added U100: MC68000_PLCC_68_PHY, Package_LCC:PLCC-68_THT-Socket, F.Cu at (254.0, 165.1)
- added U100_DIP64: MC68000_DIP_64_SOCKET, Package_DIP:DIP-64_W22.86mm_Socket_LongPads, F.Cu at (180.3, 72.4)
- added U101: ST_BLITTER_PHY, Package_LCC:PLCC-68_THT-Socket, F.Cu at (327.6, 347.2)
- added U102: EPROM_32_PINS_DIP_PHY, Package_DIP:DIP-32_W15.24mm_LongPads, F.Cu at (302.6, 421.3)
- added U103: EPROM_32_PINS_DIP_PHY, Package_DIP:DIP-32_W15.24mm_LongPads, F.Cu at (321.9, 421.3)
- added U104: LM555_TIMER_PHY, Package_DIP:DIP-8_W7.62mm_LongPads, F.Cu at (103.7, 543.7)
- added U200: MC6850_PHY, Package_DIP:DIP-24_W15.24mm_LongPads, F.Cu at (322.6, 511.5)
- added U201: MC6850_PHY, Package_DIP:DIP-24_W15.24mm_LongPads, F.Cu at (79.5, 508.3)
- added U202: YM2149_PHY, Package_DIP:DIP-40_W15.24mm_LongPads, F.Cu at (141.5, 366.9)
- added U203: MC68901_DIP_48_PHY, Package_DIP:DIP-48_W15.24mm_Socket_LongPads, F.Cu at (198.8, 345.5)
- added U204: TL497A_DIP-14_500MA_PEAK_STEP-UP_STEP-DOWN_INVERTING_SWITCH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, Package_DIP:DIP-14_W7.62mm_LongPads, F.Cu at (308.7, 321.2)
- added U205: TL497A_DIP-14_500MA_PEAK_STEP-UP_STEP-DOWN_INVERTING_SWITCH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, Package_DIP:DIP-14_W7.62mm_LongPads, F.Cu at (320.3, 321.2)
- added U206: MC1488_QUAD_LINE_EIA-232D_DRIVER_PHY, Package_DIP:DIP-14_W7.62mm_LongPads, F.Cu at (203.6, 499.1)
- added U207: MC1489_QUAD_LINE_EIA-232D_RECEIVERS_PHY, Package_DIP:DIP-14_W7.62mm_LongPads, F.Cu at (215.2, 499.1)
- added U208: PC900_PHY, Package_DIP:DIP-6_W7.62mm_LongPads, F.Cu at (301.5, 548.7)
- added U209: 74LS86_PHY, Package_DIP:DIP-14_W7.62mm_LongPads, F.Cu at (218.1, 345.4)
- added U210: 7406_PHY, Package_DIP:DIP-14_W7.62mm_LongPads, F.Cu at (322.6, 543.6)
- added U211: 74LS04_PHY, Package_DIP:DIP-14_W7.62mm_LongPads, F.Cu at (229.7, 345.4)
- added U300_DIP40: ST_DMA_DIP40_PHY, Package_DIP:DIP-40_W15.24mm_Socket_LongPads, F.Cu at (197.7, 524.6)
- added U300_PLCC44: ST_DMA_PLCC44_PHY, Package_LCC:PLCC-44_THT-Socket, F.Cu at (229.0, 528.9)
- added U301: WD1772_FLOPPY_DISK_CONTROLLER_AND_FORMATTER_PHY, Package_DIP:DIP-28_W15.24mm_LongPads, F.Cu at (153.5, 476.5)
- added U302: 74LS245_PHY, Package_DIP:DIP-20_W7.62mm_LongPads, F.Cu at (148.7, 421.3)
- added U303: 8.010613 MHz, Oscillator:Oscillator_DIP-14, F.Cu at (80.9, 552.6)
- added U304: 74LS74_PHY, Package_DIP:DIP-14_W7.62mm_LongPads, F.Cu at (79.4, 558.0)
- added U305: 7406_PHY, Package_DIP:DIP-14_W7.62mm_LongPads, F.Cu at (172.7, 496.6)
- added U306: 74LS74_PHY, Package_DIP:DIP-14_W7.62mm_LongPads, F.Cu at (171.9, 421.3)
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Routing:
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
Commit message: pcb session 2023-11-21T04:54:50+01:00 : position blitter, mounting holes
Parts:
- moved H703 536.7 mm to (360.7, 63.5)
- moved H702 507.3 mm to (203.2, 40.6)
- moved H701 498.1 mm to (78.7, 40.6)
- moved H706 414.0 mm to (360.7, 195.6)
- moved H705 352.3 mm to (203.2, 195.6)
- moved H704 347.2 mm to (78.7, 195.6)
- moved H709 347.2 mm to (360.7, 268.0)
- moved H707 280.0 mm to (78.7, 268.0)
- moved H708 279.2 mm to (203.2, 268.0)
- moved U101 233.8 mm to (166.4, 177.8), turned to -90 degrees

Commit message: pcb session 2023-11-21T05:51:32+01:00 : routing blitter north and south sides
Routing:
- net ADDR13: track 193.6 -> 371.9 mm, vias 2 -> 4
- net ADDR12: track 193.6 -> 365.0 mm, vias 2 -> 4
- net ADDR5: track 201.7 -> 368.6 mm, vias 3 -> 5
- net ADDR9: track 204.0 -> 370.9 mm, vias 3 -> 5
- net ADDR7: track 202.2 -> 369.1 mm, vias 3 -> 5
- net ADDR11: track 204.5 -> 371.4 mm, vias 3 -> 5
- net ADDR6: track 198.9 -> 362.7 mm, vias 3 -> 5
- net ADDR10: track 200.9 -> 364.8 mm, vias 3 -> 5
- net ADDR8: track 200.2 -> 364.0 mm, vias 3 -> 5
- net ADDR1: track 206.5 -> 362.3 mm, vias 3 -> 4
- net ADDR3: track 205.5 -> 358.7 mm, vias 3 -> 4
- net ADDR2: track 203.0 -> 354.3 mm, vias 3 -> 4
- net ADDR4: track 201.9 -> 350.8 mm, vias 3 -> 4
- net XLDS: track 203.0 -> 336.9 mm, vias 1 -> 2
- net RXW: track 197.4 -> 329.5 mm, vias 1 -> 2
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Other:
- board outline added: 304.8 x 243.8 mm

Commit message: pcb session 2023-11-22T23:13:50+01:00 -- place RAM, shifter and MCU
Parts:
- moved J305 276.3 mm to (129.3, 172.7), turned to 180 degrees
- moved U400 225.9 mm to (195.2, 235.1), turned to -90 degrees
- moved U602 225.8 mm to (339.1, 147.3), turned to -90 degrees
- moved U603 221.2 mm to (321.3, 147.3), turned to -90 degrees
- moved U600 219.4 mm to (348.0, 147.3), turned to -90 degrees
- moved U401 213.8 mm to (294.6, 224.8)
- moved U601 213.3 mm to (330.2, 147.3), turned to -90 degrees
Routing:
- net MDATA8: track 0.00 -> 170.6 mm, vias 0 -> 2
- net MDATA9: track 0.00 -> 163.8 mm, vias 0 -> 2
- net DATA12: track 225.3 -> 383.3 mm, vias 1 -> 3
- net DATA14: track 246.7 -> 403.4 mm, vias 2 -> 4
- net DATA13: track 249.2 -> 402.9 mm, vias 2 -> 4
- net DATA15: track 246.7 -> 397.8 mm, vias 2 -> 4
- net MDATA10: track 0.00 -> 147.6 mm, vias 0 -> 2
- net ADDR1: track 362.3 -> 509.1 mm, vias 4 -> 6
- net MDATA11: track 0.00 -> 141.0 mm, vias 0 -> 2
- net ADDR2: track 354.3 -> 493.8 mm, vias 4 -> 6
- net ADDR3: track 358.7 -> 496.7 mm, vias 4 -> 6
- net RXW: track 329.5 -> 464.0 mm, vias 2 -> 3
- net ADDR5: track 368.6 -> 501.4 mm, vias 5 -> 7
- net XCPUBG: track 254.8 -> 385.2 mm, vias 2 -> 4
- net ADDR4: track 350.8 -> 481.2 mm, vias 4 -> 6
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